File: schematics/STLINK_V2_1.kicad_sch (KiCad schematic)
At the start: 34 parts, among them J1 USB_B, J2 Conn_01x04_Socket, Q1001 S9013, X1 8MHz

Commit message: Файлы измененный Kicad
Parts:
- C0100: renamed from C1001; footprint Capacitor_SMD:C_1206_3216Metric_Pad1.33x1.80mm_HandSolder -> Capacitor_SMD:C_0805_2012Metric
- C0101: renamed from C1002; footprint Capacitor_SMD:C_1206_3216Metric_Pad1.33x1.80mm_HandSolder -> Capacitor_SMD:C_0805_2012Metric
- C0102: renamed from C1003; footprint Capacitor_SMD:C_1206_3216Metric_Pad1.33x1.80mm_HandSolder -> Capacitor_SMD:C_0805_2012Metric
- C0103: renamed from C1004; footprint Capacitor_SMD:C_1206_3216Metric_Pad1.33x1.80mm_HandSolder -> Capacitor_SMD:C_0805_2012Metric
- C0104: renamed from C1006; footprint Capacitor_SMD:C_1206_3216Metric_Pad1.33x1.80mm_HandSolder -> Capacitor_SMD:C_0805_2012Metric
- C0105: renamed from C1007; footprint Capacitor_SMD:C_1206_3216Metric_Pad1.33x1.80mm_HandSolder -> Capacitor_SMD:C_0805_2012Metric
- C1005: footprint Capacitor_SMD:C_1206_3216Metric_Pad1.33x1.80mm_HandSolder -> Capacitor_SMD:C_0805_2012Metric
- renumbered D1 to D0100, LD1002 to LD0100, LD1003 to LD0101, Q1001 to Q0100, R1008 to R0100, R1007 to R0101, R1006 to R0102, R1004 to R0103, R1003 to R0104, R1010 to R0105, R1011 to R0106, R1019 to R0107, R1018 to R0108, R1015 to R0109, R1016 to R0110, R1014 to R0111, R1009 to R0112, R1012 to R0113, R1013 to R0114, R1026 to R0115, R1025 to R0116, R1024 to R0117, R1023 to R0118, MK1 to U2, X1 to X0100
Other:
- moved on the sheet: LD0100, LD0101, R0105, R0106, R0107, R0108

Commit message: Прошелся по всей схеме: 1. почистил компоненты; 2. задал посадочные места; 3. Выставил все ссылки на плате в притык, дальнейшее расширение - смена мк
Parts:
- LD0100: value RED -> ~; footprint LED_SMD:LED_1206_3216Metric_Pad1.42x1.75mm_HandSolder -> LED_SMD:LED_0805_2012Metric
- LD0101: value GREEN -> ~; footprint LED_SMD:LED_1206_3216Metric_Pad1.42x1.75mm_HandSolder -> LED_SMD:LED_0805_2012Metric
- P0: renamed from J2; footprint (none) -> Connector_PinHeader_2.00mm:PinHeader_1x04_P2.00mm_Vertical_SMD_Pin1Left
- R0100, R0101, R0102, R0103, R0104, R0105, R0106, R0107, R0108, R0109, R0110, R0111, R0112, R0113, R0114, R0115, R0116, R0117, R0118: footprint Resistor_SMD:R_1206_3216Metric_Pad1.30x1.75mm_HandSolder -> Resistor_SMD:R_0805_2012Metric
- X0100: footprint Crystal:Crystal_HC49-U_Vertical -> Crystal:Crystal_HC49-4H_Vertical
- renumbered C1005 to C0106, J1 to USB0
Other:
- company: (none) -> Филимонов и К
Changed lines of the file:
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@@
 	(title_block
 		(date "2025-02-17")
+		(company "Филимонов и К")
 		(comment 1 "STLINK V2.1")
 		(comment 2 "Филимонов С.В.")
@@
 		(on_board yes)
 		(dnp no)
-		(property "Reference" "J2"
+		(property "Reference" "P0"
 			(at 182.88 146.0499 0)
 			(effects
@@
 			)
 		)
-		(property "Footprint" ""
+		(property "Footprint" "Connector_PinHeader_2.00mm:PinHeader_1x04_P2.00mm_Vertical_SMD_Pin1Left"
 			(at 184.15 146.05 0)
 			(effects
@@
 			(project ""
 				(path "/97e8f341-b455-4614-ab7f-cc310164e7aa/8bb2ba2e-b6e4-4843-9b9f-90d06bc3e717"
-					(reference "J2")
+					(reference "P0")
 					(unit 1)
 				)
@@
 		(dnp no)
 		(fields_autoplaced yes)
-		(property "Reference" "J1"
+		(property "Reference" "USB0"
 			(at 39.37 46.99 0)
 			(effects
@@
 			(project ""
 				(path "/97e8f341-b455-4614-ab7f-cc310164e7aa/8bb2ba2e-b6e4-4843-9b9f-90d06bc3e717"
-					(reference "J1")
+					(reference "USB0")
 					(unit 1)
 				)
@@
 			)
 		)
-		(property "Footprint" "Resistor_SMD:R_1206_3216Metric_Pad1.30x1.75mm_HandSolder"
+		(property "Footprint" "Resistor_SMD:R_0805_2012Metric"
 			(at 72.898 34.29 90)
 			(effects
@@
 			)
 		)
-		(property "Footprint" "Resistor_SMD:R_1206_3216Metric_Pad1.30x1.75mm_HandSolder"
+		(property "Footprint" "Resistor_SMD:R_0805_2012Metric"
 			(at 66.04 161.798 90)
 			(effects
@@
 			)
 		)
-		(property "Footprint" "Resistor_SMD:R_1206_3216Metric_Pad1.30x1.75mm_HandSolder"
+		(property "Footprint" "Resistor_SMD:R_0805_2012Metric"
 			(at 112.522 53.34 90)
 			(effects
@@
 			)
 		)
-		(property "Footprint" "Resistor_SMD:R_1206_3216Metric_Pad1.30x1.75mm_HandSolder"
+		(property "Footprint" "Resistor_SMD:R_0805_2012Metric"
 			(at 66.04 116.078 90)
 			(effects
@@
 			)
 		)
-		(property "Footprint" "Resistor_SMD:R_1206_3216Metric_Pad1.30x1.75mm_HandSolder"
+		(property "Footprint" "Resistor_SMD:R_0805_2012Metric"
 			(at 71.12 64.008 90)
 			(effects
@@
 			)
 		)
-		(property "Footprint" "Resistor_SMD:R_1206_3216Metric_Pad1.30x1.75mm_HandSolder"
+		(property "Footprint" "Resistor_SMD:R_0805_2012Metric"
 			(at 85.09 41.148 90)
 			(effects
@@
 			)
 		)
-		(property "Footprint" "Resistor_SMD:R_1206_3216Metric_Pad1.30x1.75mm_HandSolder"
+		(property "Footprint" "Resistor_SMD:R_0805_2012Metric"
 			(at 180.34 66.548 90)
 			(effects
@@
 			)
 		)
-		(property "Value" "RED"
+		(property "Value" "~"
 			(at 149.606 34.798 90)
 			(effects
@@
 			)
 		)
-		(property "Footprint" "LED_SMD:LED_1206_3216Metric_Pad1.42x1.75mm_HandSolder"
+		(property "Footprint" "LED_SMD:LED_0805_2012Metric"
 			(at 143.51 34.29 0)
 			(effects
@@
 			)
 		)
-		(property "Footprint" "Resistor_SMD:R_1206_3216Metric_Pad1.30x1.75mm_HandSolder"
+		(property "Footprint" "Resistor_SMD:R_0805_2012Metric"
 			(at 141.732 43.18 90)
 			(effects
@@
 			)
 		)
-		(property "Footprint" "Resistor_SMD:R_1206_3216Metric_Pad1.30x1.75mm_HandSolder"
+		(property "Footprint" "Resistor_SMD:R_0805_2012Metric"
 			(at 180.34 36.068 90)
 			(effects
@@
 			)
 		)
-		(property "Footprint" "Resistor_SMD:R_1206_3216Metric_Pad1.30x1.75mm_HandSolder"
+		(property "Footprint" "Resistor_SMD:R_0805_2012Metric"
 			(at 71.12 61.468 90)
 			(effects
@@
 			)
 		)
-		(property "Footprint" "Resistor_SMD:R_1206_3216Metric_Pad1.30x1.75mm_HandSolder"
+		(property "Footprint" "Resistor_SMD:R_0805_2012Metric"
 			(at 69.342 44.45 90)
 			(effects
@@
 			)
 		)
-		(property "Footprint" "Crystal:Crystal_HC49-U_Vertical"
+		(property "Footprint" "Crystal:Crystal_HC49-4H_Vertical"
 			(at 243.84 148.59 0)
 			(effects
@@
 			)
 		)
-		(property "Footprint" "Resistor_SMD:R_1206_3216Metric_Pad1.30x1.75mm_HandSolder"
+		(property "Footprint" "Resistor_SMD:R_0805_2012Metric"
 			(at 190.5 105.918 90)
 			(effects
@@
 			)
 		)
-		(property "Footprint" "Resistor_SMD:R_1206_3216Metric_Pad1.30x1.75mm_HandSolder"
+		(property "Footprint" "Resistor_SMD:R_0805_2012Metric"
 			(at 180.34 56.388 90)
 			(effects
@@
 			)
 		)
-		(property "Value" "GREEN"
+		(property "Value" "~"
 			(at 150.622 63.246 90)
 			(effects
@@
 			)
 		)
-		(property "Footprint" "LED_SMD:LED_1206_3216Metric_Pad1.42x1.75mm_HandSolder"
+		(property "Footprint" "LED_SMD:LED_0805_2012Metric"
 			(at 143.51 62.23 0)
 			(effects
@@
 			)
 		)
-		(property "Footprint" "Resistor_SMD:R_1206_3216Metric_Pad1.30x1.75mm_HandSolder"
+		(property "Footprint" "Resistor_SMD:R_0805_2012Metric"
 			(at 66.04 118.618 90)
 			(effects
@@
 			)
 		)
-		(property "Footprint" "Resistor_SMD:R_1206_3216Metric_Pad1.30x1.75mm_HandSolder"
+		(property "Footprint" "Resistor_SMD:R_0805_2012Metric"
 			(at 141.732 53.34 90)
 			(effects
@@
 			)
 		)
-		(property "Footprint" "Resistor_SMD:R_1206_3216Metric_Pad1.30x1.75mm_HandSolder"
+		(property "Footprint" "Resistor_SMD:R_0805_2012Metric"
 			(at 190.5 97.028 90)
 			(effects
@@
 			)
 		)
-		(property "Footprint" "Resistor_SMD:R_1206_3216Metric_Pad1.30x1.75mm_HandSolder"
+		(property "Footprint" "Resistor_SMD:R_0805_2012Metric"
 			(at 112.522 43.18 90)
 			(effects
@@
 		(on_board yes)
 		(dnp no)
-		(property "Reference" "C1005"
+		(property "Reference" "C0106"
 			(at 243.586 54.61 0)
 			(effects
@@
 			(project "stm32f4_ILI_RS_SD"
 				(path "/97e8f341-b455-4614-ab7f-cc310164e7aa/8bb2ba2e-b6e4-4843-9b9f-90d06bc3e717"
-					(reference "C1005")
+					(reference "C0106")
 					(unit 1)
 				)
@@
 			)
 		)
-		(property "Footprint" "Resistor_SMD:R_1206_3216Metric_Pad1.30x1.75mm_HandSolder"
+		(property "Footprint" "Resistor_SMD:R_0805_2012Metric"
 			(at 238.252 45.72 90)
 			(effects
@@
 			)
 		)
-		(property "Footprint" "Resistor_SMD:R_1206_3216Metric_Pad1.30x1.75mm_HandSolder"
+		(property "Footprint" "Resistor_SMD:R_0805_2012Metric"
 			(at 180.34 46.228 90)
 			(effects
