File: schematics/STM32f405RG.kicad_sch (KiCad schematic)
At the start: 15 parts, among them SW0000 Push_Button, U1 STM32F405RGTx, X0000 8MHz

Commit message: Прошелся по всей схеме: 1. почистил компоненты; 2. задал посадочные места; 3. Выставил все ссылки на плате в притык, дальнейшее расширение - смена мк
Parts:
- R0000: footprint Resistor_SMD:R_1206_3216Metric_Pad1.30x1.75mm_HandSolder -> Resistor_SMD:R_0805_2012Metric
- X0000: footprint Crystal:Crystal_HC49-U_Vertical -> Crystal:Crystal_HC49-4H_Vertical
Other:
- company: (none) -> Филимонов и К
Changed lines of the file:
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@@
 	(title_block
 		(date "2025-02-28")
+		(company "Филимонов и К")
 		(comment 1 "STM32F405RG")
 		(comment 2 "Филимонов С.В.")
@@
 			)
 		)
-		(property "Footprint" "Resistor_SMD:R_1206_3216Metric_Pad1.30x1.75mm_HandSolder"
+		(property "Footprint" "Resistor_SMD:R_0805_2012Metric"
 			(at 88.138 60.96 90)
 			(effects
@@
 			)
 		)
-		(property "Footprint" "Crystal:Crystal_HC49-U_Vertical"
+		(property "Footprint" "Crystal:Crystal_HC49-4H_Vertical"
 			(at 210.82 63.5 0)
 			(effects
