File: schematics/W25Q32_module.kicad_sch (KiCad schematic)
At the start: 6 parts, among them U7 W25Q32JVSS

Commit message: Прошелся по всей схеме: 1. почистил компоненты; 2. задал посадочные места; 3. Выставил все ссылки на плате в притык, дальнейшее расширение - смена мк
Parts:
- R0800, R0801, R0802, R0803: footprint (none) -> Resistor_SMD:R_0805_2012Metric
Other:
- company: (none) -> Филимонов и К
Changed lines of the file:
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@@
 	(title_block
 		(date "2025-02-28")
+		(company "Филимонов и К")
 		(comment 1 "Модуль памяти")
 		(comment 2 "Филимонов С.В.")
@@
 			)
 		)
-		(property "Footprint" ""
+		(property "Footprint" "Resistor_SMD:R_0805_2012Metric"
 			(at 129.54 91.948 90)
 			(effects
@@
 			)
 		)
-		(property "Footprint" ""
+		(property "Footprint" "Resistor_SMD:R_0805_2012Metric"
 			(at 129.54 89.408 90)
 			(effects
@@
 			)
 		)
-		(property "Footprint" ""
+		(property "Footprint" "Resistor_SMD:R_0805_2012Metric"
 			(at 129.54 97.028 90)
 			(effects
@@
 			)
 		)
-		(property "Footprint" ""
+		(property "Footprint" "Resistor_SMD:R_0805_2012Metric"
 			(at 129.54 94.488 90)
 			(effects

Commit message: Хмм в библиотеки был косяк
Parts:
- U7: footprint Package_SO:SOIC-8_5.23x5.23mm_P1.27mm -> Package_SO:SOIC-8_5.3x5.3mm_P1.27mm
Changed lines of the file:
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@@
 			)
 		)
-		(property "Footprint" "Package_SO:SOIC-8_5.23x5.23mm_P1.27mm"
+		(property "Footprint" "Package_SO:SOIC-8_5.3x5.3mm_P1.27mm"
 			(at 148.59 95.25 0)
 			(effects

Commit message: Множественные модификации
Parts:
- renumbered U7 to U5
Changed lines of the file:
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@@
 		(dnp no)
 		(fields_autoplaced yes)
-		(property "Reference" "U7"
+		(property "Reference" "U5"
 			(at 157.48 93.9799 0)
 			(effects
@@
 			(project ""
 				(path "/97e8f341-b455-4614-ab7f-cc310164e7aa/71095070-8281-4de7-807c-d3e17339dc65"
-					(reference "U7")
+					(reference "U5")
 					(unit 1)
 				)
