File: schematics/W5500_module.kicad_sch (KiCad schematic)
At the start: 40 parts, among them J16 RJ45_Hanrun_HR911105A_Horizon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, U7 W5500, X3 25MHz

Commit message: Файлы измененный Kicad
Parts:
- C0600: renamed from C31; footprint (none) -> Capacitor_SMD:C_0805_2012Metric
- C0601: renamed from C32; footprint (none) -> Capacitor_SMD:C_0805_2012Metric
- C0602: renamed from C30; footprint (none) -> Capacitor_SMD:C_0805_2012Metric
- C0603: renamed from C29; footprint (none) -> Capacitor_SMD:C_0805_2012Metric
- C0604: renamed from C1008; footprint Capacitor_SMD:C_1206_3216Metric_Pad1.33x1.80mm_HandSolder -> Capacitor_SMD:C_0805_2012Metric
- C0605: renamed from C1009; footprint Capacitor_SMD:C_1206_3216Metric_Pad1.33x1.80mm_HandSolder -> Capacitor_SMD:C_0805_2012Metric
- C0606: renamed from C33; footprint (none) -> Capacitor_SMD:C_0805_2012Metric
- C0607: renamed from C34; footprint (none) -> Capacitor_SMD:C_0805_2012Metric
- C0608: renamed from C35; footprint (none) -> Capacitor_SMD:C_0805_2012Metric
- C0609: renamed from C43; footprint (none) -> Capacitor_SMD:C_0805_2012Metric
- C0610: renamed from C42; footprint (none) -> Capacitor_SMD:C_0805_2012Metric
- renumbered J16 to ETH0, R42 to R0600, R43 to R0601, R44 to R0602, R45 to R0603, R46 to R0604, R47 to R0605, R14 to R0606, R17 to R0607, R19 to R0608, R18 to R0608, R20 to R0609, R21 to R0610, R31 to R0611, R32 to R0612, R23 to R0613, R33 to R0614, R22 to R0615, R34 to R0616, R13 to R0617, R37 to R0618, R38 to R0619, R39 to R0620, R40 to R0621, R41 to R0622, R35 to R0623, R36 to R0624, U7 to U5, X3 to X0600
Other:
- moved on the sheet: C0602, R0611, R0612, R0613, R0614, R0615, R0616

Commit message: Прошелся по всей схеме: 1. почистил компоненты; 2. задал посадочные места; 3. Выставил все ссылки на плате в притык, дальнейшее расширение - смена мк
Parts:
- R0600, R0601, R0602, R0603, R0604, R0605, R0606, R0607, R0608, R0609, R0610, R0611, R0612, R0613, R0614, R0615, R0616, R0617, R0618, R0619, R0620, R0621, R0622, R0623, R0624: footprint (none) -> Resistor_SMD:R_0805_2012Metric
- R0625: renamed from R0608; footprint (none) -> Resistor_SMD:R_0805_2012Metric
- X0600: footprint Crystal:Crystal_HC49-U_Vertical -> Crystal:Crystal_HC49-4H_Vertical
Other:
- company: (none) -> Филимонов и К
Changed lines of the file:
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@@
 	(title_block
 		(date "2025-02-27")
+		(company "Филимонов и К")
 		(comment 1 "W5500 модуль")
 		(comment 2 "Филимонов С.В.")
@@
 			)
 		)
-		(property "Footprint" "Crystal:Crystal_HC49-U_Vertical"
+		(property "Footprint" "Crystal:Crystal_HC49-4H_Vertical"
 			(at 86.36 138.43 0)
 			(effects
@@
 			)
 		)
-		(property "Footprint" ""
+		(property "Footprint" "Resistor_SMD:R_0805_2012Metric"
 			(at 86.36 90.678 90)
 			(effects
@@
 			)
 		)
-		(property "Footprint" ""
+		(property "Footprint" "Resistor_SMD:R_0805_2012Metric"
 			(at 86.36 95.758 90)
 			(effects
@@
 			)
 		)
-		(property "Footprint" ""
+		(property "Footprint" "Resistor_SMD:R_0805_2012Metric"
 			(at 86.36 57.658 90)
 			(effects
@@
 			)
 		)
-		(property "Footprint" ""
+		(property "Footprint" "Resistor_SMD:R_0805_2012Metric"
 			(at 179.07 130.048 90)
 			(effects
@@
 			)
 		)
-		(property "Footprint" ""
+		(property "Footprint" "Resistor_SMD:R_0805_2012Metric"
 			(at 32.512 78.74 90)
 			(effects
@@
 			)
 		)
-		(property "Footprint" ""
+		(property "Footprint" "Resistor_SMD:R_0805_2012Metric"
 			(at 86.36 65.278 90)
 			(effects
@@
 			)
 		)
-		(property "Footprint" ""
+		(property "Footprint" "Resistor_SMD:R_0805_2012Metric"
 			(at 242.57 128.778 90)
 			(effects
@@
 		(on_board yes)
 		(dnp no)
-		(property "Reference" "R0608"
+		(property "Reference" "R0625"
 			(at 78.994 90.17 90)
 			(effects
@@
 			)
 		)
-		(property "Footprint" ""
+		(property "Footprint" "Resistor_SMD:R_0805_2012Metric"
 			(at 86.36 93.218 90)
 			(effects
@@
 			(project "MasterBoard"
 				(path "/97e8f341-b455-4614-ab7f-cc310164e7aa/79d602db-a6dd-43c7-a573-120ff5d57928"
-					(reference "R0608")
+					(reference "R0625")
 					(unit 1)
 				)
@@
 			)
 		)
-		(property "Footprint" ""
+		(property "Footprint" "Resistor_SMD:R_0805_2012Metric"
 			(at 86.36 103.378 90)
 			(effects
@@
 			)
 		)
-		(property "Footprint" ""
+		(property "Footprint" "Resistor_SMD:R_0805_2012Metric"
 			(at 240.03 71.628 90)
 			(effects
@@
 			)
 		)
-		(property "Footprint" ""
+		(property "Footprint" "Resistor_SMD:R_0805_2012Metric"
 			(at 54.102 63.5 90)
 			(effects
@@
 			)
 		)
-		(property "Footprint" ""
+		(property "Footprint" "Resistor_SMD:R_0805_2012Metric"
 			(at 179.07 140.208 90)
 			(effects
@@
 			)
 		)
-		(property "Footprint" ""
+		(property "Footprint" "Resistor_SMD:R_0805_2012Metric"
 			(at 86.36 52.578 90)
 			(effects
@@
 			)
 		)
-		(property "Footprint" ""
+		(property "Footprint" "Resistor_SMD:R_0805_2012Metric"
 			(at 86.36 60.198 90)
 			(effects
@@
 			)
 		)
-		(property "Footprint" ""
+		(property "Footprint" "Resistor_SMD:R_0805_2012Metric"
 			(at 150.622 106.68 90)
 			(effects
@@
 			)
 		)
-		(property "Footprint" ""
+		(property "Footprint" "Resistor_SMD:R_0805_2012Metric"
 			(at 42.672 78.74 90)
 			(effects
@@
 			)
 		)
-		(property "Footprint" ""
+		(property "Footprint" "Resistor_SMD:R_0805_2012Metric"
 			(at 86.36 55.118 90)
 			(effects
@@
 			)
 		)
-		(property "Footprint" ""
+		(property "Footprint" "Resistor_SMD:R_0805_2012Metric"
 			(at 32.512 63.5 90)
 			(effects
@@
 			)
 		)
-		(property "Footprint" ""
+		(property "Footprint" "Resistor_SMD:R_0805_2012Metric"
 			(at 54.102 78.74 90)
 			(effects
@@
 			)
 		)
-		(property "Footprint" ""
+		(property "Footprint" "Resistor_SMD:R_0805_2012Metric"
 			(at 42.672 63.5 90)
 			(effects
@@
 			)
 		)
-		(property "Footprint" ""
+		(property "Footprint" "Resistor_SMD:R_0805_2012Metric"
 			(at 179.07 119.888 90)
 			(effects
@@
 			)
 		)
-		(property "Footprint" ""
+		(property "Footprint" "Resistor_SMD:R_0805_2012Metric"
 			(at 86.36 88.138 90)
 			(effects
@@
 			)
 		)
-		(property "Footprint" ""
+		(property "Footprint" "Resistor_SMD:R_0805_2012Metric"
 			(at 240.03 61.468 90)
 			(effects
@@
 			)
 		)
-		(property "Footprint" ""
+		(property "Footprint" "Resistor_SMD:R_0805_2012Metric"
 			(at 242.57 118.618 90)
 			(effects
@@
 			)
 		)
-		(property "Footprint" ""
+		(property "Footprint" "Resistor_SMD:R_0805_2012Metric"
 			(at 86.36 98.298 90)
 			(effects
@@
 			)
 		)
-		(property "Footprint" ""
+		(property "Footprint" "Resistor_SMD:R_0805_2012Metric"
 			(at 86.36 62.738 90)
 			(effects

Commit message: Множественные модификации
Parts:
- renumbered U5 to U4
Changed lines of the file:
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@@
 		(dnp no)
 		(fields_autoplaced yes)
-		(property "Reference" "U5"
+		(property "Reference" "U4"
 			(at 115.1733 43.18 0)
 			(effects
@@
 			(project ""
 				(path "/97e8f341-b455-4614-ab7f-cc310164e7aa/79d602db-a6dd-43c7-a573-120ff5d57928"
-					(reference "U5")
+					(reference "U4")
 					(unit 1)
 				)
