File: schematics/EndStop.kicad_sch (KiCad schematic)
At the start: 3 parts, among them J22 Conn_01x03

Commit message: Файлы измененный Kicad
Parts:
- C0900: renamed from C205; footprint Capacitor_SMD:C_1206_3216Metric_Pad1.33x1.80mm_HandSolder -> Capacitor_SMD:C_0805_2012Metric
- ES00: renamed from J22; value Conn_01x03 -> JST_XH_B3B
- renumbered R213 to R0900
Changed lines of the file:
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@@
 		(dnp no)
 		(fields_autoplaced yes)
-		(property "Reference" "J?"
+		(property "Reference" "ES00"
 			(at 151.13 92.7099 0)
 			(effects
@@
 			)
 		)
-		(property "Value" "Conn_01x03"
+		(property "Value" "JST_XH_B3B"
 			(at 151.13 95.2499 0)
 			(effects
@@
 			(project "MasterBoard"
 				(path "/97e8f341-b455-4614-ab7f-cc310164e7aa/0020857d-77ad-4b1f-afb2-65480b85c325"
-					(reference "J22")
+					(reference "ES06")
 					(unit 1)
 				)
 				(path "/97e8f341-b455-4614-ab7f-cc310164e7aa/15b1724a-2f36-4aa6-bc5e-02dcfe1e0071"
-					(reference "J21")
+					(reference "ES05")
 					(unit 1)
 				)
 				(path "/97e8f341-b455-4614-ab7f-cc310164e7aa/2cb344d1-bc6a-4ba0-9e7f-cb68bc3ab9dc"
-					(reference "J20")
+					(reference "J04")
 					(unit 1)
 				)
 				(path "/97e8f341-b455-4614-ab7f-cc310164e7aa/4e2e899a-7a0c-4669-897b-8dedbdd1b4ee"
-					(reference "J18")
+					(reference "JES02")
 					(unit 1)
 				)
 				(path "/97e8f341-b455-4614-ab7f-cc310164e7aa/94ff1a88-0c2a-40cb-bd19-cf6a210b21bd"
-					(reference "J19")
+					(reference "ES03")
 					(unit 1)
 				)
 				(path "/97e8f341-b455-4614-ab7f-cc310164e7aa/a1fd2dac-a455-4c85-b79b-43aa768602d3"
-					(reference "J17")
+					(reference "ES01")
 					(unit 1)
 				)
 				(path "/97e8f341-b455-4614-ab7f-cc310164e7aa/c32cc6e0-b940-4ade-a351-c5b9da254a31"
-					(reference "J?")
+					(reference "ES00")
 					(unit 1)
 				)
@@
 		(dnp no)
 		(fields_autoplaced yes)
-		(property "Reference" "C205"
+		(property "Reference" "C0900"
 			(at 134.62 95.2499 0)
 			(effects
@@
 			)
 		)
-		(property "Footprint" "Capacitor_SMD:C_1206_3216Metric_Pad1.33x1.80mm_HandSolder"
+		(property "Footprint" "Capacitor_SMD:C_0805_2012Metric"
 			(at 129.8448 92.71 0)
 			(effects
@@
 			(project "MasterBoard"
 				(path "/97e8f341-b455-4614-ab7f-cc310164e7aa/0020857d-77ad-4b1f-afb2-65480b85c325"
-					(reference "C211")
+					(reference "C0906")
 					(unit 1)
 				)
 				(path "/97e8f341-b455-4614-ab7f-cc310164e7aa/15b1724a-2f36-4aa6-bc5e-02dcfe1e0071"
-					(reference "C210")
+					(reference "C0905")
 					(unit 1)
 				)
 				(path "/97e8f341-b455-4614-ab7f-cc310164e7aa/2cb344d1-bc6a-4ba0-9e7f-cb68bc3ab9dc"
-					(reference "C209")
+					(reference "C0904")
 					(unit 1)
 				)
 				(path "/97e8f341-b455-4614-ab7f-cc310164e7aa/4e2e899a-7a0c-4669-897b-8dedbdd1b4ee"
-					(reference "C207")
+					(reference "C0902")
 					(unit 1)
 				)
 				(path "/97e8f341-b455-4614-ab7f-cc310164e7aa/94ff1a88-0c2a-40cb-bd19-cf6a210b21bd"
-					(reference "C208")
+					(reference "C0903")
 					(unit 1)
 				)
 				(path "/97e8f341-b455-4614-ab7f-cc310164e7aa/a1fd2dac-a455-4c85-b79b-43aa768602d3"
-					(reference "C206")
+					(reference "C0901")
 					(unit 1)
 				)
 				(path "/97e8f341-b455-4614-ab7f-cc310164e7aa/c32cc6e0-b940-4ade-a351-c5b9da254a31"
-					(reference "C205")
+					(reference "C0900")
 					(unit 1)
 				)
@@
 		(on_board yes)
 		(dnp no)
-		(property "Reference" "R213"
+		(property "Reference" "R0900"
 			(at 135.382 84.582 0)
 			(effects
@@
 			(project "MasterBoard"
 				(path "/97e8f341-b455-4614-ab7f-cc310164e7aa/0020857d-77ad-4b1f-afb2-65480b85c325"
-					(reference "R219")
+					(reference "R0906")
 					(unit 1)
 				)
 				(path "/97e8f341-b455-4614-ab7f-cc310164e7aa/15b1724a-2f36-4aa6-bc5e-02dcfe1e0071"
-					(reference "R218")
+					(reference "R0905")
 					(unit 1)
 				)
 				(path "/97e8f341-b455-4614-ab7f-cc310164e7aa/2cb344d1-bc6a-4ba0-9e7f-cb68bc3ab9dc"
-					(reference "R217")
+					(reference "R0904")
 					(unit 1)
 				)
 				(path "/97e8f341-b455-4614-ab7f-cc310164e7aa/4e2e899a-7a0c-4669-897b-8dedbdd1b4ee"
-					(reference "R215")
+					(reference "R0902")
 					(unit 1)
 				)
 				(path "/97e8f341-b455-4614-ab7f-cc310164e7aa/94ff1a88-0c2a-40cb-bd19-cf6a210b21bd"
-					(reference "R216")
+					(reference "R0903")
 					(unit 1)
 				)
 				(path "/97e8f341-b455-4614-ab7f-cc310164e7aa/a1fd2dac-a455-4c85-b79b-43aa768602d3"
-					(reference "R214")
+					(reference "R0901")
 					(unit 1)
 				)
 				(path "/97e8f341-b455-4614-ab7f-cc310164e7aa/c32cc6e0-b940-4ade-a351-c5b9da254a31"
-					(reference "R213")
-					(unit 1)
-				)
+					(reference "R0900")
+					(unit 1)
+				)

Commit message: Прошелся по всей схеме: 1. почистил компоненты; 2. задал посадочные места; 3. Выставил все ссылки на плате в притык, дальнейшее расширение - смена мк
Parts:
- R0900: footprint Resistor_SMD:R_1206_3216Metric_Pad1.30x1.75mm_HandSolder -> Resistor_SMD:R_0805_2012Metric
Other:
- company: (none) -> Филимонов и К
Changed lines of the file:
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@@
 	(title_block
 		(date "2025-02-27")
+		(company "Филимонов и К")
 		(comment 1 "Концевик")
 		(comment 2 "Филимонов С.В.")
@@
 			)
 		)
-		(property "Footprint" "Resistor_SMD:R_1206_3216Metric_Pad1.30x1.75mm_HandSolder"
+		(property "Footprint" "Resistor_SMD:R_0805_2012Metric"
 			(at 132.588 86.36 90)
 			(effects
