File: schematics/power.kicad_sch (KiCad schematic)
At the start: 41 parts, among them U10 LM2596S-ADJ, U11 LM2596S-ADJ, U12 RT9193-33GB, U9 LM2596S-ADJ

Commit message: Множественные модификации
Parts:
- PWR0: footprint Connector_Phoenix_MC:PhoenixContact_MC_1,5_2-G-3.81_1x02_P3.81mm_Horizontal -> Connector_PinHeader_2.54mm:KLS2
- renumbered U12 to U10, U9 to U7, U10 to U8, U11 to U9
Changed lines of the file:
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@@
 		(dnp no)
 		(fields_autoplaced yes)
-		(property "Reference" "U9"
+		(property "Reference" "U7"
 			(at 86.36 36.83 0)
 			(effects
@@
 			(project ""
 				(path "/97e8f341-b455-4614-ab7f-cc310164e7aa/7330fb6d-3de7-4c19-a7a3-dd8fb4865426"
-					(reference "U9")
+					(reference "U7")
 					(unit 1)
 				)
@@
 		(dnp no)
 		(fields_autoplaced yes)
-		(property "Reference" "U11"
+		(property "Reference" "U9"
 			(at 92.71 129.54 0)
 			(effects
@@
 			(project "MasterBoard"
 				(path "/97e8f341-b455-4614-ab7f-cc310164e7aa/7330fb6d-3de7-4c19-a7a3-dd8fb4865426"
-					(reference "U11")
+					(reference "U9")
 					(unit 1)
 				)
@@
 		(dnp no)
 		(fields_autoplaced yes)
-		(property "Reference" "U12"
+		(property "Reference" "U10"
 			(at 205.74 34.29 0)
 			(effects
@@
 			(project "MasterBoard"
 				(path "/97e8f341-b455-4614-ab7f-cc310164e7aa/7330fb6d-3de7-4c19-a7a3-dd8fb4865426"
-					(reference "U12")
+					(reference "U10")
 					(unit 1)
 				)
@@
 			)
 		)
-		(property "Footprint" "Connector_Phoenix_MC:PhoenixContact_MC_1,5_2-G-3.81_1x02_P3.81mm_Horizontal"
+		(property "Footprint" "Connector_PinHeader_2.54mm:KLS2"
 			(at 212.09 91.44 0)
 			(effects
@@
 		(dnp no)
 		(fields_autoplaced yes)
-		(property "Reference" "U10"
+		(property "Reference" "U8"
 			(at 86.36 69.85 0)
 			(effects
@@
 			(project "MasterBoard"
 				(path "/97e8f341-b455-4614-ab7f-cc310164e7aa/7330fb6d-3de7-4c19-a7a3-dd8fb4865426"
-					(reference "U10")
+					(reference "U8")
 					(unit 1)
 				)

Commit message: Был косяк в обозначениях
Parts:
- PWR0: footprint Connector_PinHeader_2.54mm:KLS2 -> Library:KLS2
Changed lines of the file:
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@@
 			)
 		)
-		(property "Footprint" "Connector_PinHeader_2.54mm:KLS2"
+		(property "Footprint" "Library:KLS2"
 			(at 212.09 91.44 0)
 			(effects
