File: schematics/power.kicad_sch (KiCad schematic)
At the start: 41 parts, among them U10 RT9193-33GB, U7 LM2596S-ADJ, U8 LM2596S-ADJ, U9 LM2596S-ADJ

Commit message: Множественные обновления схем
Other:
- company: Филимонов и К -> (none)
- title: (none) -> OctopusNode
Changed lines of the file:
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@@
 	(paper "A4")
 	(title_block
-		(company "Филимонов и К")
+		(title "OctopusNode")
 		(comment 1 "Питание")
 		(comment 2 "Филимонов С.В.")

Commit message: Обновил обозначения, а то старая нумерация была специфической
Parts:
- renumbered C9900 to C1, C9909 to C10, C9910 to C11, C9911 to C12, C9912 to C13, C9913 to C14, C9903 to C2, C9906 to C3, C9901 to C4, C9904 to C5, C9907 to C6, C9908 to C7, C9902 to C8, C9905 to C9, D9900 to D2, D9901 to D3, D9902 to D4, L9900 to L1, L9901 to L2, L9902 to L3, LD9900 to LD1, LD9901 to LD2, LD9902 to LD3, LD9903 to LD4, PWR0 to PWR1, R9900 to R1, R9909 to R10, R9910 to R11, R9911 to R12, R9903 to R2, R9906 to R3, R9901 to R4, R9904 to R5, R9907 to R6, R9902 to R7, R9905 to R8, R9908 to R9, U7 to U1, U8 to U2, U9 to U3, U10 to U4

Commit message: Правки схем, возможно что-то было не корректно выбрано
Parts:
- C1, C2, C3, C4, C5, C6: footprint Capacitor_SMD:C_0805_2012Metric -> Capacitor_SMD:CP_Elec_6.3x7.7
Connections:
- net +24V: now also PWR1.2 (Pin_2); no longer PWR1.1 (Pin_1)
- net GND: now also PWR1.1 (Pin_1); no longer PWR1.2 (Pin_2)
Changed lines of the file:
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@@
 			)
 		)
-		(property "Footprint" "Capacitor_SMD:C_0805_2012Metric"
+		(property "Footprint" "Capacitor_SMD:CP_Elec_6.3x7.7"
 			(at 63.1952 54.61 0)
 			(effects
@@
 	(symbol
 		(lib_id "Connector_Generic:Conn_01x02")
-		(at 212.09 91.44 0)
+		(at 212.09 93.98 0)
+		(mirror x)
 		(unit 1)
 		(exclude_from_sim no)
@@
 		(on_board yes)
 		(dnp no)
-		(fields_autoplaced yes)
 		(property "Reference" "PWR1"
-			(at 214.63 91.4399 0)
+			(at 214.63 93.9801 0)
 			(effects
 				(font
@@
 		)
 		(property "Value" "Conn_01x02"
-			(at 214.63 93.9799 0)
+			(at 214.63 91.4401 0)
 			(effects
 				(font
@@
 		)
 		(property "Footprint" "Library:KLS2"
-			(at 212.09 91.44 0)
+			(at 212.09 93.98 0)
 			(effects
 				(font
@@
 		)
 		(property "Datasheet" "~"
-			(at 212.09 91.44 0)
+			(at 212.09 93.98 0)
 			(effects
 				(font
@@
 		)
 		(property "Description" "Generic connector, single row, 01x02, script generated (kicad-library-utils/schlib/autogen/connector/)"
-			(at 212.09 91.44 0)
+			(at 212.09 93.98 0)
 			(effects
 				(font
@@
 			)
 		)
-		(property "Footprint" "Capacitor_SMD:C_0805_2012Metric"
+		(property "Footprint" "Capacitor_SMD:CP_Elec_6.3x7.7"
 			(at 63.1952 87.63 0)
 			(effects
@@
 			)
 		)
-		(property "Footprint" "Capacitor_SMD:C_0805_2012Metric"
+		(property "Footprint" "Capacitor_SMD:CP_Elec_6.3x7.7"
 			(at 119.0752 152.4 0)
 			(effects
@@
 			)
 		)
-		(property "Footprint" "Capacitor_SMD:C_0805_2012Metric"
+		(property "Footprint" "Capacitor_SMD:CP_Elec_6.3x7.7"
 			(at 69.5452 147.32 0)
 			(effects
@@
 			)
 		)
-		(property "Footprint" "Capacitor_SMD:C_0805_2012Metric"
+		(property "Footprint" "Capacitor_SMD:CP_Elec_6.3x7.7"
 			(at 112.7252 59.69 0)
 			(effects
@@
 			)
 		)
-		(property "Footprint" "Capacitor_SMD:C_0805_2012Metric"
+		(property "Footprint" "Capacitor_SMD:CP_Elec_6.3x7.7"
 			(at 112.7252 92.71 0)
 			(effects
