File: schematics/STM32F407VG.kicad_sch (KiCad schematic)
At the start: 15 parts, among them X2 8MHz

Commit message: Добавил кнопку на сброс
Parts:
- removed R2: 0, Resistor_SMD:R_1206_3216Metric_Pad1.30x1.75mm_HandSolder, symbol Device:R
- added C31, C32: 100n, Capacitor_SMD:C_1206_3216Metric_Pad1.33x1.80mm_HandSolder, symbol Device:C
- added C33: 100n, Capacitor_SMD:C_0805_2012Metric, symbol Device:C
- added R746: 10k, Resistor_SMD:R_0805_2012Metric, symbol Device:R
- added SW1: SW_DPST_x2, Button_Switch_SMD:SW_SPST_PTS647_Sx38, symbol Switch:SW_DPST_x2
- C9: value 1u -> 4.7u
Connections:
- net +3.3V: now also C3.1, C4.1, C5.1, C6.1, C7.1, C8.1, C31.1, C32.1, R746.2, SW1.2 (B)
- net GND: now also R1.2, C31.2, C32.2, C33.2; no longer R1.1
- net NRST: now also C33.1, R746.1, SW1.1 (A)
- net at MK2.94 (BOOT0): now also R1.1; no longer R1.2
Other:
- moved on the sheet: C1, C2, C3, C4, C5, C6, C7, C8, C9, R1, X2
