File: MasterBoard.kicad_pcb (KiCad board)
At the start: 2 copper layers, 0 parts

Commit message: Выгрузил элементы в трассировщик, модели все подгружены, настал этап трассировки платы
Parts:
- added C0000: 100n, Capacitor_SMD:C_0805_2012Metric, F.Cu at (394.9, 71.0)
- added C0001: 2.2u, Capacitor_SMD:C_0805_2012Metric, F.Cu at (394.9, 74.0)
- added C0002: 2.2u, Capacitor_SMD:C_0805_2012Metric, F.Cu at (394.9, 77.0)
- added C0003: 100n, Capacitor_SMD:C_0805_2012Metric, F.Cu at (394.9, 80.0)
- added C0004: 100n, Capacitor_SMD:C_0805_2012Metric, F.Cu at (394.9, 83.0)
- added C0005: 100n, Capacitor_SMD:C_0805_2012Metric, F.Cu at (394.9, 86.0)
- added C0006: 100n, Capacitor_SMD:C_0805_2012Metric, F.Cu at (399.4, 71.0)
- added C0007: 100n, Capacitor_SMD:C_0805_2012Metric, F.Cu at (399.4, 74.0)
- added C0008: 1u, Capacitor_SMD:C_0805_2012Metric, F.Cu at (399.4, 77.0)
- added C0009: 20p, Capacitor_SMD:C_0805_2012Metric, F.Cu at (399.4, 80.0)
- added C0010: 20p, Capacitor_SMD:C_0805_2012Metric, F.Cu at (399.4, 83.0)
- added C0100: 100n, Capacitor_SMD:C_0805_2012Metric, F.Cu at (330.2, 111.1)
- added C0101: 100n, Capacitor_SMD:C_0805_2012Metric, F.Cu at (330.2, 114.1)
- added C0102: 100n, Capacitor_SMD:C_0805_2012Metric, F.Cu at (330.2, 117.1)
- added C0103: 100n, Capacitor_SMD:C_0805_2012Metric, F.Cu at (330.2, 120.1)
- added C0104: 20p, Capacitor_SMD:C_0805_2012Metric, F.Cu at (330.2, 123.1)
- added C0105: 20p, Capacitor_SMD:C_0805_2012Metric, F.Cu at (330.2, 126.1)
- added C0106: 100n, Capacitor_SMD:C_0805_2012Metric, F.Cu at (330.2, 129.2)
- added C0200: 100n, Capacitor_SMD:C_0805_2012Metric, F.Cu at (380.1, 88.6)
- added C0201: 4.7u, Capacitor_SMD:C_0805_2012Metric, F.Cu at (380.1, 91.6)
- added C0202: 10u, Capacitor_SMD:C_0805_2012Metric, F.Cu at (380.1, 94.6)
- added C0203: 100n, Capacitor_SMD:C_0805_2012Metric, F.Cu at (380.1, 97.6)
- added C0300: 100n, Capacitor_SMD:C_0805_2012Metric, F.Cu at (437.0, 82.8)
- added C0500: 100n, Capacitor_SMD:C_0805_2012Metric, F.Cu at (374.0, 115.4)
- added C0600: 10n, Capacitor_SMD:C_0805_2012Metric, F.Cu at (343.3, 50.9)
- added C0601: 4.7u, Capacitor_SMD:C_0805_2012Metric, F.Cu at (343.3, 53.9)
- added C0602: 100n, Capacitor_SMD:C_0805_2012Metric, F.Cu at (343.3, 57.0)
- added C0603: 100n, Capacitor_SMD:C_0805_2012Metric, F.Cu at (343.3, 60.0)
- added C0604: 18p, Capacitor_SMD:C_0805_2012Metric, F.Cu at (343.3, 63.0)
- added C0605: 18p, Capacitor_SMD:C_0805_2012Metric, F.Cu at (343.3, 66.0)
- added C0606: 100n, Capacitor_SMD:C_0805_2012Metric, F.Cu at (347.8, 50.9)
- added C0607: 22n, Capacitor_SMD:C_0805_2012Metric, F.Cu at (347.8, 53.9)
- added C0608: 6.8n, Capacitor_SMD:C_0805_2012Metric, F.Cu at (347.8, 57.0)
- added C0609: 10n, Capacitor_SMD:C_0805_2012Metric, F.Cu at (347.8, 60.0)
- added C0610: 6.8n, Capacitor_SMD:C_0805_2012Metric, F.Cu at (347.8, 63.0)
- added C0700: 10u, Capacitor_SMD:C_0805_2012Metric, F.Cu at (330.2, 71.0)
- added C0701: 10n, Capacitor_SMD:C_0805_2012Metric, F.Cu at (330.2, 74.0)
- added C0702: 10n, Capacitor_SMD:C_0805_2012Metric, F.Cu at (330.2, 77.0)
- added C0703: 1u, Capacitor_SMD:C_0805_2012Metric, F.Cu at (330.2, 80.0)
- added C0704: 1u, Capacitor_SMD:C_0805_2012Metric, F.Cu at (330.2, 83.0)
- added C0705: 1u, Capacitor_SMD:C_0805_2012Metric, F.Cu at (330.2, 86.0)
- added C0706: 18p, Capacitor_SMD:C_0805_2012Metric, F.Cu at (330.2, 89.0)
- added C0707: 18p, Capacitor_SMD:C_0805_2012Metric, F.Cu at (330.2, 92.1)
- added C0800: 10u, Capacitor_SMD:C_0805_2012Metric, F.Cu at (374.0, 143.2)
- added C0900: 10u, Capacitor_SMD:C_0805_2012Metric, F.Cu at (344.1, 152.8)
- added C0901: 10u, Capacitor_SMD:C_0805_2012Metric, F.Cu at (330.2, 152.8)
- added C0902: 10u, Capacitor_SMD:C_0805_2012Metric, F.Cu at (394.9, 152.1)
- added C0903: 10u, Capacitor_SMD:C_0805_2012Metric, F.Cu at (408.9, 152.1)
- added C0904: 10u, Capacitor_SMD:C_0805_2012Metric, F.Cu at (437.6, 152.1)
- added C0905: 10u, Capacitor_SMD:C_0805_2012Metric, F.Cu at (423.7, 152.1)
- added C1000: 100u, Capacitor_SMD:CP_Elec_6.3x7.7, F.Cu at (443.0, 123.5)
- added C1001: 100u, Capacitor_SMD:C_0805_2012Metric, F.Cu at (440.0, 137.9)
- added C1002: 100u, Capacitor_SMD:CP_Elec_6.3x7.7, F.Cu at (414.2, 123.5)
- added C1003: 100u, Capacitor_SMD:C_0805_2012Metric, F.Cu at (411.2, 137.9)
- added C1004: 100u, Capacitor_SMD:CP_Elec_6.3x7.7, F.Cu at (443.0, 100.1)
- added C1005: 100u, Capacitor_SMD:C_0805_2012Metric, F.Cu at (440.0, 114.5)
- added C1006: 100u, Capacitor_SMD:CP_Elec_6.3x7.7, F.Cu at (414.2, 100.1)
- added C1007: 100u, Capacitor_SMD:C_0805_2012Metric, F.Cu at (411.2, 114.5)
- added C9900: 100u, Capacitor_SMD:C_0805_2012Metric, F.Cu at (397.7, 27.6)
- added C9901: 220u, Capacitor_SMD:C_0805_2012Metric, F.Cu at (397.7, 30.6)
- added C9902: 10n, Capacitor_SMD:C_0805_2012Metric, F.Cu at (397.7, 33.6)
- added C9903: 100u, Capacitor_SMD:C_0805_2012Metric, F.Cu at (397.7, 36.6)
- added C9904: 220u, Capacitor_SMD:C_0805_2012Metric, F.Cu at (397.7, 39.6)
- added C9905: 10n, Capacitor_SMD:C_0805_2012Metric, F.Cu at (402.2, 27.6)
- added C9906: 100u, Capacitor_SMD:C_0805_2012Metric, F.Cu at (402.2, 30.6)
- added C9907: 220u, Capacitor_SMD:C_0805_2012Metric, F.Cu at (402.2, 33.6)
- added C9908: 10n, Capacitor_SMD:C_0805_2012Metric, F.Cu at (402.2, 36.6)
- added C9909: 1u, Capacitor_SMD:C_0805_2012Metric, F.Cu at (402.2, 39.6)
- added C9910: 100n, Capacitor_SMD:C_0805_2012Metric, F.Cu at (406.6, 27.6)
- added C9911: 22n, Capacitor_SMD:C_0805_2012Metric, F.Cu at (406.6, 30.6)
- added C9912: 10u, Capacitor_SMD:C_0805_2012Metric, F.Cu at (406.6, 33.6)
- added C9913: 100n, Capacitor_SMD:C_0805_2012Metric, F.Cu at (406.6, 36.6)
- added D0100: BAT60A, Diode_SMD:D_SOD-323, F.Cu at (339.5, 138.4)
- added D0200: BAT60A, Diode_SMD:D_SOD-323, F.Cu at (384.5, 94.6)
- added D9900: 1N5822, PCM_4ms_Diode:D_DO-214AC_SMA, F.Cu at (389.1, 53.0)
- added D9901: 1N5822, PCM_4ms_Diode:D_DO-214AC_SMA, F.Cu at (389.1, 57.3)
- added D9902: 1N5822, PCM_4ms_Diode:D_DO-214AC_SMA, F.Cu at (389.1, 61.7)
- added DISP0: IDC-14, Connector_IDC:IDC-Header_2x07_P2.54mm_Vertical, F.Cu at (442.5, 32.2)
- added ES00: JST_XH_B3B, Connector_JST:JST_XH_B3B-XH-A_1x03_P2.50mm_Vertical, F.Cu at (345.4, 146.9)
- added ES01: JST_XH_B3B, Connector_JST:JST_XH_B3B-XH-A_1x03_P2.50mm_Vertical, F.Cu at (331.4, 146.9)
- added ES03: JST_XH_B3B, Connector_JST:JST_XH_B3B-XH-A_1x03_P2.50mm_Vertical, F.Cu at (410.1, 146.2)
- added ES05: JST_XH_B3B, Connector_JST:JST_XH_B3B-XH-A_1x03_P2.50mm_Vertical, F.Cu at (424.9, 146.2)
- added ETH0: RJ45_Hanrun_HR911105A_Horizontal, Connector_RJ:RJ45_Hanrun_HR911105A_Horizontal, F.Cu at (333.5, 31.1)
- added ETH1: RJ45_Hanrun_HR911105A_Horizontal, Connector_RJ:RJ45_Hanrun_HR911105A_Horizontal, F.Cu at (338.0, 74.5)
- added FAN0: Fan_CPU_4pin, Connector:FanPinHeader_1x04_P2.54mm_Vertical, F.Cu at (369.6, 122.6)
- added HOTEND0: IDC-16, Connector_IDC:IDC-Header_2x08_P2.54mm_Vertical, F.Cu at (430.5, 32.2)
- added J04: JST_XH_B3B, Connector_JST:JST_XH_B3B-XH-A_1x03_P2.50mm_Vertical, F.Cu at (438.9, 146.2)
- added J10: WF-2, Library:WF-2, F.Cu at (375.5, 110.8)
- added JES02: JST_XH_B3B, Connector_JST:JST_XH_B3B-XH-A_1x03_P2.50mm_Vertical, F.Cu at (396.2, 146.2)
- added JP0: SolderJumper_3_Open, Jumper:SolderJumper-3_P1.3mm_Open_RoundedPad1.0x1.5mm, F.Cu at (440.6, 134.4)
- added JP1: ~, Connector_PinHeader_1.00mm:PinHeader_1x02_P1.00mm_Vertical, F.Cu at (445.1, 137.1)
- added JP1001: ~, Connector_PinHeader_1.00mm:PinHeader_1x03_P1.00mm_Vertical, F.Cu at (439.5, 129.1)
- added JP1002: ~, Connector_PinHeader_1.00mm:PinHeader_1x03_P1.00mm_Vertical, F.Cu at (442.8, 129.1)
- added JP1003: ~, Connector_PinHeader_1.00mm:PinHeader_1x03_P1.00mm_Vertical, F.Cu at (446.2, 129.1)
- added JP1004: ~, Connector_PinHeader_1.00mm:PinHeader_1x03_P1.00mm_Vertical, F.Cu at (410.7, 129.1)
- added JP1005: ~, Connector_PinHeader_1.00mm:PinHeader_1x03_P1.00mm_Vertical, F.Cu at (414.0, 129.1)
- added JP1006: ~, Connector_PinHeader_1.00mm:PinHeader_1x03_P1.00mm_Vertical, F.Cu at (417.4, 129.1)
- added JP1007: ~, Connector_PinHeader_1.00mm:PinHeader_1x03_P1.00mm_Vertical, F.Cu at (439.5, 105.7)
- added JP1008: ~, Connector_PinHeader_1.00mm:PinHeader_1x03_P1.00mm_Vertical, F.Cu at (442.8, 105.7)
- added JP1009: ~, Connector_PinHeader_1.00mm:PinHeader_1x03_P1.00mm_Vertical, F.Cu at (446.2, 105.7)
- added JP1010: ~, Connector_PinHeader_1.00mm:PinHeader_1x03_P1.00mm_Vertical, F.Cu at (410.7, 105.7)
- added JP1011: ~, Connector_PinHeader_1.00mm:PinHeader_1x03_P1.00mm_Vertical, F.Cu at (414.0, 105.7)
- added JP1012: ~, Connector_PinHeader_1.00mm:PinHeader_1x03_P1.00mm_Vertical, F.Cu at (417.4, 105.7)
- added JP2: SolderJumper_3_Open, Jumper:SolderJumper-3_P1.3mm_Open_RoundedPad1.0x1.5mm, F.Cu at (411.8, 134.4)
- added JP3: ~, Connector_PinHeader_1.00mm:PinHeader_1x02_P1.00mm_Vertical, F.Cu at (416.3, 137.1)
- added JP4: SolderJumper_3_Open, Jumper:SolderJumper-3_P1.3mm_Open_RoundedPad1.0x1.5mm, F.Cu at (440.6, 111.0)
- added JP5: ~, Connector_PinHeader_1.00mm:PinHeader_1x02_P1.00mm_Vertical, F.Cu at (445.1, 113.7)
- added JP6: SolderJumper_3_Open, Jumper:SolderJumper-3_P1.3mm_Open_RoundedPad1.0x1.5mm, F.Cu at (411.8, 111.0)
- added JP7: ~, Connector_PinHeader_1.00mm:PinHeader_1x02_P1.00mm_Vertical, F.Cu at (416.3, 113.7)
- added L0700: 10u, Inductor_SMD:L_1206_3216Metric, F.Cu at (361.7, 94.6)
- added L9900: 33u, Inductor_SMD:L_APV_APH0650, F.Cu at (390.5, 30.2)
- added L9901: 33u, Inductor_SMD:L_APV_APH0650, F.Cu at (390.5, 38.4)
- added L9902: 33u, Inductor_SMD:L_APV_APH0650, F.Cu at (390.5, 46.7)
- added LD0100: ~, LED_SMD:LED_0805_2012Metric, F.Cu at (330.2, 132.2)
- added LD0101: ~, LED_SMD:LED_0805_2012Metric, F.Cu at (330.2, 135.2)
- added LD0200: ~, LED_SMD:LED_0805_2012Metric, F.Cu at (384.6, 88.6)
- added LD0201: ~, LED_SMD:LED_0805_2012Metric, F.Cu at (384.6, 91.6)
- added LD0500: ~, LED_SMD:LED_0805_2012Metric, F.Cu at (381.0, 113.7)
- added LD9900: ~, LED_SMD:LED_0805_2012Metric, F.Cu at (397.8, 54.4)
- added LD9901: ~, LED_SMD:LED_0805_2012Metric, F.Cu at (397.8, 57.5)
- added LD9902: ~, LED_SMD:LED_0805_2012Metric, F.Cu at (397.8, 60.5)
- added LD9903: ~, LED_SMD:LED_0805_2012Metric, F.Cu at (397.8, 63.6)
- added M0: ~, Library:MotorSocket, F.Cu at (429.6, 130.1)
- added M1: ~, Library:MotorSocket, F.Cu at (400.8, 130.1)
- added M2: ~, Library:MotorSocket, F.Cu at (429.6, 106.7)
- added M3: ~, Library:MotorSocket, F.Cu at (400.8, 106.7)
- added OE0: M3, Connector_JST:JST_XH_B4B-XH-A_1x04_P2.50mm_Vertical, F.Cu at (414.3, 29.4)
- added OX0: M0, Connector_JST:JST_XH_B4B-XH-A_1x04_P2.50mm_Vertical, F.Cu at (414.3, 37.2)
- added OY0: M1, Connector_JST:JST_XH_B4B-XH-A_1x04_P2.50mm_Vertical, F.Cu at (414.3, 45.0)
- added OZ0: M2, Connector_JST:JST_XH_B4B-XH-A_1x04_P2.50mm_Vertical, F.Cu at (414.3, 52.9)
- added OZ1: M2, Connector_JST:JST_XH_B4B-XH-A_1x04_P2.50mm_Vertical, F.Cu at (414.3, 60.6)
- added P0: Conn_01x04_Socket, Connector_PinHeader_2.00mm:PinHeader_1x04_P2.00mm_Vertical_SMD_Pin1Left, F.Cu at (360.4, 132.2)
- added Q0100: S9013, Package_TO_SOT_SMD:SOT-23, F.Cu at (334.8, 139.3)
- added Q0500: 2N7002, PCM_4ms_Package_SOT:SOT-23, F.Cu at (380.9, 110.0)
- added R0000: 100k, Resistor_SMD:R_0805_2012Metric, F.Cu at (403.8, 92.1)
- added R0100: 10k, Resistor_SMD:R_0805_2012Metric, F.Cu at (334.6, 111.1)
- added R0101: 100, Resistor_SMD:R_0805_2012Metric, F.Cu at (334.6, 114.0)
- added R0102: 36k, Resistor_SMD:R_0805_2012Metric, F.Cu at (334.6, 117.0)
- added R0103: 10, Resistor_SMD:R_0805_2012Metric, F.Cu at (334.6, 119.9)
- added R0104: 10, Resistor_SMD:R_0805_2012Metric, F.Cu at (334.6, 122.9)
- added R0105: 4.7k, Resistor_SMD:R_0805_2012Metric, F.Cu at (334.6, 125.8)
- added R0106: 4.7k, Resistor_SMD:R_0805_2012Metric, F.Cu at (334.6, 128.8)
- added R0107: 1k, Resistor_SMD:R_0805_2012Metric, F.Cu at (339.0, 111.1)
- added R0108: 1k, Resistor_SMD:R_0805_2012Metric, F.Cu at (339.0, 114.0)
- added R0109: 10k, Resistor_SMD:R_0805_2012Metric, F.Cu at (339.0, 117.0)
- added R0110: 10k, Resistor_SMD:R_0805_2012Metric, F.Cu at (339.0, 119.9)
- added R0111: 100, Resistor_SMD:R_0805_2012Metric, F.Cu at (339.0, 122.9)
- added R0112: 100k, Resistor_SMD:R_0805_2012Metric, F.Cu at (339.0, 125.8)
- added R0113: 100k, Resistor_SMD:R_0805_2012Metric, F.Cu at (339.0, 128.8)
- added R0114: 100k, Resistor_SMD:R_0805_2012Metric, F.Cu at (343.4, 111.1)
- added R0115: 22, Resistor_SMD:R_0805_2012Metric, F.Cu at (343.4, 114.0)
- added R0116: 22, Resistor_SMD:R_0805_2012Metric, F.Cu at (343.4, 117.0)
- added R0117: 22, Resistor_SMD:R_0805_2012Metric, F.Cu at (343.4, 119.9)
- added R0118: 22, Resistor_SMD:R_0805_2012Metric, F.Cu at (343.4, 122.9)
- added R0200: 1k, Resistor_SMD:R_0805_2012Metric, F.Cu at (388.5, 71.0)
- added R0201: 1k, Resistor_SMD:R_0805_2012Metric, F.Cu at (388.5, 73.9)
- added R0202: 1k, Resistor_SMD:R_0805_2012Metric, F.Cu at (388.5, 76.9)
- added R0203: 1k, Resistor_SMD:R_0805_2012Metric, F.Cu at (388.5, 79.8)
- added R0204: 10k, Resistor_SMD:R_0805_2012Metric, F.Cu at (388.5, 82.8)
- added R0300: 10, Resistor_SMD:R_0805_2012Metric, F.Cu at (437.0, 71.0)
- added R0301: 10, Resistor_SMD:R_0805_2012Metric, F.Cu at (437.0, 73.9)
- added R0302: 10, Resistor_SMD:R_0805_2012Metric, F.Cu at (437.0, 76.9)
- added R0303: 10, Resistor_SMD:R_0805_2012Metric, F.Cu at (437.0, 79.8)
- added R0400: -, Resistor_SMD:R_0805_2012Metric, F.Cu at (369.6, 128.4)
- added R0401: -, Resistor_SMD:R_0805_2012Metric, F.Cu at (369.6, 131.3)
- added R0500: 1k, Resistor_SMD:R_0805_2012Metric, F.Cu at (369.6, 102.6)
- added R0501: 1k, Resistor_SMD:R_0805_2012Metric, F.Cu at (369.6, 105.5)
- added R0502: 10k, Resistor_SMD:R_0805_2012Metric, F.Cu at (369.6, 108.5)
- added R0503: 10k, Connector_JST:JST_PH_B2B-PH-K_1x02_P2.00mm_Vertical, F.Cu at (374.7, 103.8)
- added R0504: 10k, Resistor_SMD:R_0805_2012Metric, F.Cu at (369.6, 111.5)
- added R0600: 10, Resistor_SMD:R_0805_2012Metric, F.Cu at (350.2, 27.6)
- added R0601: 10, Resistor_SMD:R_0805_2012Metric, F.Cu at (350.2, 30.5)
- added R0602: 10, Resistor_SMD:R_0805_2012Metric, F.Cu at (350.2, 33.5)
- added R0603: 10, Resistor_SMD:R_0805_2012Metric, F.Cu at (350.2, 36.4)
- added R0604: 10, Resistor_SMD:R_0805_2012Metric, F.Cu at (350.2, 39.4)
- added R0605: 10, Resistor_SMD:R_0805_2012Metric, F.Cu at (350.2, 42.3)
- added R0606: 10k, Resistor_SMD:R_0805_2012Metric, F.Cu at (350.2, 45.2)
- added R0607: 10k, Resistor_SMD:R_0805_2012Metric, F.Cu at (354.6, 27.6)
- added R0608: 10k, Resistor_SMD:R_0805_2012Metric, F.Cu at (354.6, 30.5)
- added R0609: 10k, Resistor_SMD:R_0805_2012Metric, F.Cu at (354.6, 33.5)
- added R0610: 10k, Resistor_SMD:R_0805_2012Metric, F.Cu at (354.6, 36.4)
- added R0611: 10k, Resistor_SMD:R_0805_2012Metric, F.Cu at (354.6, 39.4)
- added R0612: 10k, Resistor_SMD:R_0805_2012Metric, F.Cu at (354.6, 42.3)
- added R0613: 10k, Resistor_SMD:R_0805_2012Metric, F.Cu at (354.6, 45.2)
- added R0614: 10k, Resistor_SMD:R_0805_2012Metric, F.Cu at (359.0, 27.6)
- added R0615: 10k, Resistor_SMD:R_0805_2012Metric, F.Cu at (359.0, 30.5)
- added R0616: 10k, Resistor_SMD:R_0805_2012Metric, F.Cu at (359.0, 33.5)
- added R0617: 12.4k, Resistor_SMD:R_0805_2012Metric, F.Cu at (359.0, 36.4)
- added R0618: 51, Resistor_SMD:R_0805_2012Metric, F.Cu at (359.0, 39.4)
- added R0619: 51, Resistor_SMD:R_0805_2012Metric, F.Cu at (359.0, 42.3)
- added R0620: 10, Resistor_SMD:R_0805_2012Metric, F.Cu at (359.0, 45.2)
- added R0621: 82, Resistor_SMD:R_0805_2012Metric, F.Cu at (363.4, 27.6)
- added R0622: 82, Resistor_SMD:R_0805_2012Metric, F.Cu at (363.4, 30.5)
- added R0623: 10k, Resistor_SMD:R_0805_2012Metric, F.Cu at (363.4, 33.5)
- added R0624: 10k, Resistor_SMD:R_0805_2012Metric, F.Cu at (363.4, 36.4)
- added R0625: 10k, Resistor_SMD:R_0805_2012Metric, F.Cu at (363.4, 39.4)
- added R0700: 10, Resistor_SMD:R_0805_2012Metric, F.Cu at (334.6, 100.2)
- added R0701: 10, Resistor_SMD:R_0805_2012Metric, F.Cu at (334.6, 103.2)
- added R0702: 10, Resistor_SMD:R_0805_2012Metric, F.Cu at (334.6, 106.1)
- added R0703: 10, Resistor_SMD:R_0805_2012Metric, F.Cu at (339.0, 94.3)
- added R0704: 10, Resistor_SMD:R_0805_2012Metric, F.Cu at (339.0, 97.3)
- added R0705: 10, Resistor_SMD:R_0805_2012Metric, F.Cu at (339.0, 100.2)
- added R0706: 2.7k, Resistor_SMD:R_0805_2012Metric, F.Cu at (339.0, 103.2)
- added R0707: 50, Resistor_SMD:R_0805_2012Metric, F.Cu at (339.0, 106.1)
- added R0708: 50, Resistor_SMD:R_0805_2012Metric, F.Cu at (343.4, 94.3)
- added R0709: 50, Resistor_SMD:R_0805_2012Metric, F.Cu at (343.4, 97.3)
- added R0710: 50, Resistor_SMD:R_0805_2012Metric, F.Cu at (343.4, 100.2)
- added R0800: 10, Resistor_SMD:R_0805_2012Metric, F.Cu at (369.6, 136.3)
- added R0801: 10, Resistor_SMD:R_0805_2012Metric, F.Cu at (369.6, 139.2)
- added R0802: 10, Resistor_SMD:R_0805_2012Metric, F.Cu at (369.6, 142.2)
- added R0803: 10, Resistor_SMD:R_0805_2012Metric, F.Cu at (369.6, 145.1)
- added R0900: 10k, Resistor_SMD:R_0805_2012Metric, F.Cu at (348.6, 152.8)
- added R0901: 10k, Resistor_SMD:R_0805_2012Metric, F.Cu at (334.6, 152.8)
- added R0902: 10k, Resistor_SMD:R_0805_2012Metric, F.Cu at (399.3, 152.1)
- added R0903: 10k, Resistor_SMD:R_0805_2012Metric, F.Cu at (413.3, 152.1)
- added R0904: 10k, Resistor_SMD:R_0805_2012Metric, F.Cu at (442.1, 152.1)
- added R0905: 10k, Resistor_SMD:R_0805_2012Metric, F.Cu at (428.1, 152.1)
- added R1000: 22k, Resistor_SMD:R_0805_2012Metric, F.Cu at (445.7, 134.1)
- added R1001: 22k, Resistor_SMD:R_0805_2012Metric, F.Cu at (416.9, 134.1)
- added R1002: 22k, Resistor_SMD:R_0805_2012Metric, F.Cu at (445.7, 110.7)
- added R1003: 22k, Resistor_SMD:R_0805_2012Metric, F.Cu at (416.9, 110.7)
- added R48: 1k, Resistor_SMD:R_0805_2012Metric, F.Cu at (334.6, 94.3)
- added R49: 1k, Resistor_SMD:R_0805_2012Metric, F.Cu at (334.6, 97.3)
- added R9800: 1k, Resistor_SMD:R_0805_2012Metric, F.Cu at (439.5, 61.6)
- added R9900: 1.2k, Resistor_SMD:R_0805_2012Metric, F.Cu at (397.7, 42.6)
- added R9901: 500, Resistor_SMD:R_0805_2012Metric, F.Cu at (397.7, 45.5)
- added R9902: 10k, Resistor_SMD:R_0805_2012Metric, F.Cu at (397.7, 48.5)
- added R9903: 1.2k, Resistor_SMD:R_0805_2012Metric, F.Cu at (397.7, 51.5)
- added R9904: 500, Resistor_SMD:R_0805_2012Metric, F.Cu at (402.1, 42.6)
- added R9905: 10k, Resistor_SMD:R_0805_2012Metric, F.Cu at (402.1, 45.5)
- added R9906: 3k, Resistor_SMD:R_0805_2012Metric, F.Cu at (402.1, 48.5)
- added R9907: 1k, Resistor_SMD:R_0805_2012Metric, F.Cu at (402.1, 51.5)
- added R9908: 1k, Resistor_SMD:R_0805_2012Metric, F.Cu at (406.5, 42.6)
- added R9909: 1k, Resistor_SMD:R_0805_2012Metric, F.Cu at (406.5, 45.5)
- added R9910: 1k, Resistor_SMD:R_0805_2012Metric, F.Cu at (406.5, 48.5)
- added R9911: 1k, Resistor_SMD:R_0805_2012Metric, F.Cu at (406.5, 51.5)
- added SD0: Micro_SD_Card, Connector_Card:microSD_HC_Hirose_DM3AT-SF-PEJM5, F.Cu at (426.4, 78.8)
- added SW0000: Push_Button, Button_Switch_SMD:SW_SPST_PTS647_Sx38, F.Cu at (396.9, 90.8)
- added U1: STM32F405RGTx, Package_QFP:LQFP-64_10x10mm_P0.5mm, F.Cu at (408.8, 76.7)
- added U10: LM2596S-ADJ, PCM_Package_TO_SOT_SMD_AKL:TO-263-5_TabPin3_ThermalVias, F.Cu at (376.6, 44.9)
- added U11: LM2596S-ADJ, PCM_Package_TO_SOT_SMD_AKL:TO-263-5_TabPin3_ThermalVias, F.Cu at (376.6, 57.4)
- added U12: RT9193-33GB, Package_TO_SOT_SMD:SOT-23-5, F.Cu at (402.5, 55.3)
- added U2: STM32F103CBTx, Package_QFP:LQFP-48_7x7mm_P0.5mm, F.Cu at (351.3, 132.8)
- added U3: FT232RL, Package_SO:SSOP-28_5.3x10.2mm_P0.65mm, F.Cu at (372.6, 93.1)
- added U5: W5500, Package_QFP:LQFP-48_7x7mm_P0.5mm, F.Cu at (333.6, 61.8)
- added U6: ENC28J60x-SO, Package_SO:SOIC-28W_7.5x17.9mm_P1.27mm, F.Cu at (358.9, 79.3)
- added U7: W25Q32JVSS, Package_SO:SOIC-8_5.3x5.3mm_P1.27mm, F.Cu at (376.9, 138.2)
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
Commit message: Решил отказатся от платы Ender
Parts:
- removed C0000, C0003, C0004, C0005, C0006, C0007, C0100, C0101, C0102, C0103, C0106, C0200, C0203, C0300, C0500, C0602, C0603, C0606, C9910, C9913: 100n, Capacitor_SMD:C_0805_2012Metric
- removed C0001, C0002: 2.2u, Capacitor_SMD:C_0805_2012Metric
- removed C0008, C0703, C0704, C0705, C9909: 1u, Capacitor_SMD:C_0805_2012Metric
- removed C0009, C0010, C0104, C0105: 20p, Capacitor_SMD:C_0805_2012Metric
- removed C0201, C0601: 4.7u, Capacitor_SMD:C_0805_2012Metric
- removed C0202, C0700, C0800, C0900, C0901, C0902, C0903, C0904, C0905, C9912: 10u, Capacitor_SMD:C_0805_2012Metric
- removed C0600, C0609, C0701, C0702, C9902, C9905, C9908: 10n, Capacitor_SMD:C_0805_2012Metric
- removed C0604, C0605, C0706, C0707: 18p, Capacitor_SMD:C_0805_2012Metric
- removed C0607, C9911: 22n, Capacitor_SMD:C_0805_2012Metric
- removed C0608, C0610: 6.8n, Capacitor_SMD:C_0805_2012Metric
- removed C1000, C1002, C1004, C1006: 100u, Capacitor_SMD:CP_Elec_6.3x7.7
- removed C1001, C1003, C1005, C1007, C9900, C9903, C9906: 100u, Capacitor_SMD:C_0805_2012Metric
- removed C9901, C9904, C9907: 220u, Capacitor_SMD:C_0805_2012Metric
- removed D0100, D0200: BAT60A, Diode_SMD:D_SOD-323
- removed D9900, D9901, D9902: 1N5822, PCM_4ms_Diode:D_DO-214AC_SMA
- removed DISP0: IDC-14, Connector_IDC:IDC-Header_2x07_P2.54mm_Vertical
- removed ES00, ES01, ES03, ES05, J04, JES02: JST_XH_B3B, Connector_JST:JST_XH_B3B-XH-A_1x03_P2.50mm_Vertical
- removed ETH0, ETH1: RJ45_Hanrun_HR911105A_Horizontal, Connector_RJ:RJ45_Hanrun_HR911105A_Horizontal
- removed FAN0: Fan_CPU_4pin, Connector:FanPinHeader_1x04_P2.54mm_Vertical
- removed HOTEND0: IDC-16, Connector_IDC:IDC-Header_2x08_P2.54mm_Vertical
- removed J10: WF-2, Library:WF-2
- removed JP0, JP2, JP4, JP6: SolderJumper_3_Open, Jumper:SolderJumper-3_P1.3mm_Open_RoundedPad1.0x1.5mm
- removed JP1, JP3, JP5, JP7: ~, Connector_PinHeader_1.00mm:PinHeader_1x02_P1.00mm_Vertical
- removed JP1001, JP1002, JP1003, JP1004, JP1005, JP1006, JP1007, JP1008, JP1009, JP1010, JP1011, JP1012: ~, Connector_PinHeader_1.00mm:PinHeader_1x03_P1.00mm_Vertical
- removed L0700: 10u, Inductor_SMD:L_1206_3216Metric
- removed L9900, L9901, L9902: 33u, Inductor_SMD:L_APV_APH0650
- removed LD0100, LD0101, LD0200, LD0201, LD0500, LD9900, LD9901, LD9902, LD9903: ~, LED_SMD:LED_0805_2012Metric
- removed M0, M1, M2, M3: ~, Library:MotorSocket
- removed OE0: M3, Connector_JST:JST_XH_B4B-XH-A_1x04_P2.50mm_Vertical
- removed OX0: M0, Connector_JST:JST_XH_B4B-XH-A_1x04_P2.50mm_Vertical
- removed OY0: M1, Connector_JST:JST_XH_B4B-XH-A_1x04_P2.50mm_Vertical
- removed OZ0, OZ1: M2, Connector_JST:JST_XH_B4B-XH-A_1x04_P2.50mm_Vertical
- removed P0: Conn_01x04_Socket, Connector_PinHeader_2.00mm:PinHeader_1x04_P2.00mm_Vertical_SMD_Pin1Left
- removed Q0100: S9013, Package_TO_SOT_SMD:SOT-23
- removed Q0500: 2N7002, PCM_4ms_Package_SOT:SOT-23
- removed R0000, R0112, R0113, R0114: 100k, Resistor_SMD:R_0805_2012Metric
- removed R0100, R0109, R0110, R0204, R0502, R0504, R0606, R0607, R0608, R0609, R0610, R0611, R0612, R0613, R0614, R0615, R0616, R0623, R0624, R0625, R0900, R0901, R0902, R0903, R0904, R0905, R9902, R9905: 10k, Resistor_SMD:R_0805_2012Metric
- removed R0101, R0111: 100, Resistor_SMD:R_0805_2012Metric
- removed R0102: 36k, Resistor_SMD:R_0805_2012Metric
- removed R0103, R0104, R0300, R0301, R0302, R0303, R0600, R0601, R0602, R0603, R0604, R0605, R0620, R0700, R0701, R0702, R0703, R0704, R0705, R0800, R0801, R0802, R0803: 10, Resistor_SMD:R_0805_2012Metric
- removed R0105, R0106: 4.7k, Resistor_SMD:R_0805_2012Metric
- removed R0107, R0108, R0200, R0201, R0202, R0203, R0500, R0501, R48, R49, R9800, R9907, R9908, R9909, R9910, R9911: 1k, Resistor_SMD:R_0805_2012Metric
- removed R0115, R0116, R0117, R0118: 22, Resistor_SMD:R_0805_2012Metric
- removed R0400, R0401: -, Resistor_SMD:R_0805_2012Metric
- removed R0503: 10k, Connector_JST:JST_PH_B2B-PH-K_1x02_P2.00mm_Vertical
- removed R0617: 12.4k, Resistor_SMD:R_0805_2012Metric
- removed R0618, R0619: 51, Resistor_SMD:R_0805_2012Metric
- removed R0621, R0622: 82, Resistor_SMD:R_0805_2012Metric
- removed R0706: 2.7k, Resistor_SMD:R_0805_2012Metric
- removed R0707, R0708, R0709, R0710: 50, Resistor_SMD:R_0805_2012Metric
- removed R1000, R1001, R1002, R1003: 22k, Resistor_SMD:R_0805_2012Metric
- removed R9900, R9903: 1.2k, Resistor_SMD:R_0805_2012Metric
- removed R9901, R9904: 500, Resistor_SMD:R_0805_2012Metric
- removed R9906: 3k, Resistor_SMD:R_0805_2012Metric
- removed SD0: Micro_SD_Card, Connector_Card:microSD_HC_Hirose_DM3AT-SF-PEJM5
- removed SW0000: Push_Button, Button_Switch_SMD:SW_SPST_PTS647_Sx38
- removed U1: STM32F405RGTx, Package_QFP:LQFP-64_10x10mm_P0.5mm
- removed U10, U11, U9: LM2596S-ADJ, PCM_Package_TO_SOT_SMD_AKL:TO-263-5_TabPin3_ThermalVias
- removed U12: RT9193-33GB, Package_TO_SOT_SMD:SOT-23-5
- removed U2: STM32F103CBTx, Package_QFP:LQFP-48_7x7mm_P0.5mm
- removed U3: FT232RL, Package_SO:SSOP-28_5.3x10.2mm_P0.65mm
- removed U5: W5500, Package_QFP:LQFP-48_7x7mm_P0.5mm
- removed U6: ENC28J60x-SO, Package_SO:SOIC-28W_7.5x17.9mm_P1.27mm
- removed U7: W25Q32JVSS, Package_SO:SOIC-8_5.3x5.3mm_P1.27mm
- removed U8: CD4066BPW, Package_SO:TSSOP-14_4.4x5mm_P0.65mm
- removed USB0, USB1: USB_B, Connector_USB:USB_B_OST_USB-B1HSxx_Horizontal
- removed X0000, X0100: 8MHz, Crystal:Crystal_HC49-4H_Vertical
- removed X0600, X0700: 25MHz, Crystal:Crystal_HC49-4H_Vertical

Commit message: Начал делать трассировку
Parts:
- added C0000: 100n, Capacitor_SMD:C_0805_2012Metric, F.Cu at (100.1, 103.0)
- added C0001: 2.2u, Capacitor_SMD:C_0805_2012Metric, F.Cu at (100.1, 106.0)
- added C0002: 2.2u, Capacitor_SMD:C_0805_2012Metric, F.Cu at (100.1, 109.0)
- added C0003: 100n, Capacitor_SMD:C_0805_2012Metric, F.Cu at (100.1, 112.0)
- added C0004: 100n, Capacitor_SMD:C_0805_2012Metric, F.Cu at (100.1, 115.0)
- added C0005: 100n, Capacitor_SMD:C_0805_2012Metric, F.Cu at (100.1, 118.0)
- added C0006: 100n, Capacitor_SMD:C_0805_2012Metric, F.Cu at (104.6, 103.0)
- added C0007: 100n, Capacitor_SMD:C_0805_2012Metric, F.Cu at (104.6, 106.0)
- added C0008: 1u, Capacitor_SMD:C_0805_2012Metric, F.Cu at (104.6, 109.0)
- added C0009: 20p, Capacitor_SMD:C_0805_2012Metric, F.Cu at (104.6, 112.0)
- added C0010: 20p, Capacitor_SMD:C_0805_2012Metric, F.Cu at (104.6, 115.0)
- added C0200: 100n, Capacitor_SMD:C_0805_2012Metric, F.Cu at (381.4, 33.6)
- added C0201: 4.7u, Capacitor_SMD:C_0805_2012Metric, F.Cu at (381.4, 36.6)
- added C0202: 10u, Capacitor_SMD:C_0805_2012Metric, F.Cu at (381.4, 39.6)
- added C0203: 100n, Capacitor_SMD:C_0805_2012Metric, F.Cu at (381.4, 42.6)
- added C0500: 100n, Capacitor_SMD:C_0805_2012Metric, F.Cu at (207.0, 96.1)
- added C0600: 10n, Capacitor_SMD:C_0805_2012Metric, F.Cu at (113.3, 82.9)
- added C0601: 4.7u, Capacitor_SMD:C_0805_2012Metric, F.Cu at (113.3, 85.9)
- added C0602: 100n, Capacitor_SMD:C_0805_2012Metric, F.Cu at (113.3, 88.9)
- added C0603: 100n, Capacitor_SMD:C_0805_2012Metric, F.Cu at (113.3, 91.9)
- added C0604: 18p, Capacitor_SMD:C_0805_2012Metric, F.Cu at (113.3, 95.0)
- added C0605: 18p, Capacitor_SMD:C_0805_2012Metric, F.Cu at (113.3, 98.0)
- added C0606: 100n, Capacitor_SMD:C_0805_2012Metric, F.Cu at (117.7, 82.9)
- added C0607: 22n, Capacitor_SMD:C_0805_2012Metric, F.Cu at (117.7, 85.9)
- added C0608: 6.8n, Capacitor_SMD:C_0805_2012Metric, F.Cu at (117.7, 88.9)
- added C0609: 10n, Capacitor_SMD:C_0805_2012Metric, F.Cu at (117.7, 91.9)
- added C0610: 6.8n, Capacitor_SMD:C_0805_2012Metric, F.Cu at (117.7, 95.0)
- added C0800: 10u, Capacitor_SMD:C_0805_2012Metric, F.Cu at (202.5, 108.0)
- added C0900: 10u, Capacitor_SMD:C_0805_2012Metric, F.Cu at (313.1, 175.7)
- added C0901: 10u, Capacitor_SMD:C_0805_2012Metric, F.Cu at (322.3, 160.6)
- added C0902: 10u, Capacitor_SMD:C_0805_2012Metric, F.Cu at (342.0, 174.1)
- added C0903: 10u, Capacitor_SMD:C_0805_2012Metric, F.Cu at (308.3, 160.6)
- added C0904: 10u, Capacitor_SMD:C_0805_2012Metric, F.Cu at (328.0, 174.1)
- added C0905: 10u, Capacitor_SMD:C_0805_2012Metric, F.Cu at (336.6, 161.2)
- added C1000: 100u, Capacitor_SMD:CP_Elec_6.3x7.7, F.Cu at (277.9, 14.0)
- added C1001: 100u, Capacitor_SMD:C_0805_2012Metric, B.Cu at (278.0, 11.4)
- added C1002: 100u, Capacitor_SMD:CP_Elec_6.3x7.7, F.Cu at (298.3, 13.9)
- added C1003: 100u, Capacitor_SMD:C_0805_2012Metric, B.Cu at (298.4, 11.4)
- added C1004: 100u, Capacitor_SMD:CP_Elec_6.3x7.7, F.Cu at (318.9, 13.9)
- added C1005: 100u, Capacitor_SMD:C_0805_2012Metric, B.Cu at (318.9, 11.4)
- added C1006: 100u, Capacitor_SMD:CP_Elec_6.3x7.7, F.Cu at (339.5, 13.9)
- added C1007: 100u, Capacitor_SMD:C_0805_2012Metric, B.Cu at (339.5, 11.4)
- added C9900: 100u, Capacitor_SMD:C_0805_2012Metric, F.Cu at (168.4, 15.3)
- added C9901: 220u, Capacitor_SMD:C_0805_2012Metric, F.Cu at (168.4, 18.3)
- added C9902: 10n, Capacitor_SMD:C_0805_2012Metric, F.Cu at (168.4, 21.3)
- added C9903: 100u, Capacitor_SMD:C_0805_2012Metric, F.Cu at (168.4, 24.4)
- added C9904: 220u, Capacitor_SMD:C_0805_2012Metric, F.Cu at (168.4, 27.4)
- added C9905: 10n, Capacitor_SMD:C_0805_2012Metric, F.Cu at (172.8, 15.3)
- added C9906: 100u, Capacitor_SMD:C_0805_2012Metric, F.Cu at (172.8, 18.3)
- added C9907: 220u, Capacitor_SMD:C_0805_2012Metric, F.Cu at (172.8, 21.3)
- added C9908: 10n, Capacitor_SMD:C_0805_2012Metric, F.Cu at (172.8, 24.4)
- added C9909: 1u, Capacitor_SMD:C_0805_2012Metric, F.Cu at (172.8, 27.4)
- added C9910: 100n, Capacitor_SMD:C_0805_2012Metric, F.Cu at (177.3, 15.3)
- added C9911: 22n, Capacitor_SMD:C_0805_2012Metric, F.Cu at (177.3, 18.3)
- added C9912: 10u, Capacitor_SMD:C_0805_2012Metric, F.Cu at (177.3, 21.3)
- added C9913: 100n, Capacitor_SMD:C_0805_2012Metric, F.Cu at (177.3, 24.4)
- added D0200: BAT60A, Diode_SMD:D_SOD-323, B.Cu at (357.1, 10.6)
- added D9800: BAT60A, Diode_SMD:D_SOD-323, F.Cu at (118.9, 51.9)
- added D9900: 1N5822, PCM_4ms_Diode:D_DO-214AC_SMA, F.Cu at (159.7, 40.7)
- added D9901: 1N5822, PCM_4ms_Diode:D_DO-214AC_SMA, F.Cu at (159.7, 45.1)
- added D9902: 1N5822, PCM_4ms_Diode:D_DO-214AC_SMA, F.Cu at (159.7, 49.5)
- added DISP0: IDC-14, Connector_IDC:IDC-Header_2x07_P2.54mm_Vertical, F.Cu at (129.6, 19.9)
- added ES00: JST_XH_B3B, Connector_JST:JST_XH_B3B-XH-A_1x03_P2.50mm_Vertical, F.Cu at (314.3, 169.8)
- added ES01: JST_XH_B3B, Connector_JST:JST_XH_B3B-XH-A_1x03_P2.50mm_Vertical, F.Cu at (323.5, 154.7)
- added ES02: JST_XH_B3B, Connector_JST:JST_XH_B3B-XH-A_1x03_P2.50mm_Vertical, F.Cu at (343.2, 168.1)
- added ES03: JST_XH_B3B, Connector_JST:JST_XH_B3B-XH-A_1x03_P2.50mm_Vertical, F.Cu at (309.6, 154.7)
- added ES04: JST_XH_B3B, Connector_JST:JST_XH_B3B-XH-A_1x03_P2.50mm_Vertical, F.Cu at (329.3, 168.1)
- added ES05: JST_XH_B3B, Connector_JST:JST_XH_B3B-XH-A_1x03_P2.50mm_Vertical, F.Cu at (337.8, 155.2)
- added ETH0: RJ45_Hanrun_HR911105A_Horizontal, Connector_RJ:RJ45_Hanrun_HR911105A_Horizontal, F.Cu at (345.7, 100.4)
- added FAN0: Fan_CPU_4pin, Connector:FanPinHeader_1x04_P2.54mm_Vertical, F.Cu at (125.5, 105.2)
- added HOTEND0: IDC-16, Connector_IDC:IDC-Header_2x08_P2.54mm_Vertical, F.Cu at (117.6, 19.9)
- added J10: WF-2, Library:WF-2, F.Cu at (204.0, 91.5)
- added JP0: SolderJumper_3_Open, Jumper:SolderJumper-3_P1.3mm_Open_RoundedPad1.0x1.5mm, B.Cu at (287.2, 22.8)
- added JP1: ~, Connector_PinHeader_2.54mm:PinHeader_1x02_P2.54mm_Vertical, F.Cu at (283.7, 16.4)
- added JP1001: ~, Connector_PinHeader_2.54mm:PinHeader_1x03_P2.54mm_Vertical, F.Cu at (289.4, 16.4)
- added JP1002: ~, Connector_PinHeader_2.54mm:PinHeader_1x03_P2.54mm_Vertical, F.Cu at (286.6, 16.4)
- added JP1003: ~, Connector_PinHeader_2.54mm:PinHeader_1x03_P2.54mm_Vertical, F.Cu at (292.2, 16.4)
- added JP1004: ~, Connector_PinHeader_2.54mm:PinHeader_1x03_P2.54mm_Vertical, F.Cu at (309.9, 16.4)
- added JP1005: ~, Connector_PinHeader_2.54mm:PinHeader_1x03_P2.54mm_Vertical, F.Cu at (307.1, 16.4)
- added JP1006: ~, Connector_PinHeader_2.54mm:PinHeader_1x03_P2.54mm_Vertical, F.Cu at (312.6, 16.4)
- added JP1007: ~, Connector_PinHeader_2.54mm:PinHeader_1x03_P2.54mm_Vertical, F.Cu at (330.4, 16.4)
- added JP1008: ~, Connector_PinHeader_2.54mm:PinHeader_1x03_P2.54mm_Vertical, F.Cu at (327.6, 16.4)
- added JP1009: ~, Connector_PinHeader_2.54mm:PinHeader_1x03_P2.54mm_Vertical, F.Cu at (333.2, 16.4)
- added JP1010: ~, Connector_PinHeader_2.54mm:PinHeader_1x03_P2.54mm_Vertical, F.Cu at (350.9, 16.4)
- added JP1011: ~, Connector_PinHeader_2.54mm:PinHeader_1x03_P2.54mm_Vertical, F.Cu at (348.1, 16.4)
- added JP1012: ~, Connector_PinHeader_2.54mm:PinHeader_1x03_P2.54mm_Vertical, F.Cu at (353.8, 16.4)
- added JP2: SolderJumper_3_Open, Jumper:SolderJumper-3_P1.3mm_Open_RoundedPad1.0x1.5mm, B.Cu at (307.7, 22.8)
- added JP3: ~, Connector_PinHeader_2.54mm:PinHeader_1x02_P2.54mm_Vertical, F.Cu at (304.2, 16.4)
- added JP4: SolderJumper_3_Open, Jumper:SolderJumper-3_P1.3mm_Open_RoundedPad1.0x1.5mm, B.Cu at (328.2, 22.9)
- added JP5: ~, Connector_PinHeader_2.54mm:PinHeader_1x02_P2.54mm_Vertical, F.Cu at (324.8, 16.4)
- added JP6: SolderJumper_3_Open, Jumper:SolderJumper-3_P1.3mm_Open_RoundedPad1.0x1.5mm, B.Cu at (348.8, 22.9)
- added JP7: ~, Connector_PinHeader_2.54mm:PinHeader_1x02_P2.54mm_Vertical, F.Cu at (345.4, 16.4)
- added L9900: 33u, Inductor_SMD:L_APV_APH0650, F.Cu at (161.2, 17.9)
- added L9901: 33u, Inductor_SMD:L_APV_APH0650, F.Cu at (161.2, 26.2)
- added L9902: 33u, Inductor_SMD:L_APV_APH0650, F.Cu at (161.2, 34.4)
- added LD0200: ~, LED_SMD:LED_0805_2012Metric, F.Cu at (364.8, 3.56)
- added LD0201: ~, LED_SMD:LED_0805_2012Metric, F.Cu at (362.7, 3.56)
- added LD0500: ~, LED_SMD:LED_0805_2012Metric, F.Cu at (202.6, 96.1)
- added LD9900: ~, LED_SMD:LED_0805_2012Metric, F.Cu at (168.4, 42.2)
- added LD9901: ~, LED_SMD:LED_0805_2012Metric, F.Cu at (168.4, 45.2)
- added LD9902: ~, LED_SMD:LED_0805_2012Metric, F.Cu at (168.4, 48.3)
- added LD9903: ~, LED_SMD:LED_0805_2012Metric, F.Cu at (168.4, 51.3)
- added M0: ~, Library:MotorSocket, F.Cu at (283.4, 14.2)
- added M1: ~, Library:MotorSocket, F.Cu at (303.9, 14.2)
- added M2: ~, Library:MotorSocket, F.Cu at (324.4, 14.2)
- added M3: ~, Library:MotorSocket, F.Cu at (344.9, 14.1)
- added OE0: M3, Connector_JST:JST_XH_B4B-XH-A_1x04_P2.50mm_Vertical, F.Cu at (344.2, 2.52)
- added OX0: M0, Connector_JST:JST_XH_B4B-XH-A_1x04_P2.50mm_Vertical, F.Cu at (279.7, 2.52)
- added OY0: M1, Connector_JST:JST_XH_B4B-XH-A_1x04_P2.50mm_Vertical, F.Cu at (299.4, 2.52)
- added OZ0: M2, Connector_JST:JST_XH_B4B-XH-A_1x04_P2.50mm_Vertical, F.Cu at (314.3, 2.52)
- added OZ1: M2, Connector_JST:JST_XH_B4B-XH-A_1x04_P2.50mm_Vertical, F.Cu at (329.2, 2.52)
- added PWR0: Conn_01x02, Library:KLS2, F.Cu at (122.5, 153.7)
- added Q0500: 2N7002, PCM_4ms_Package_SOT:SOT-23, F.Cu at (206.1, 84.2)
- added R0000: 100k, Resistor_SMD:R_0805_2012Metric, F.Cu at (109.0, 124.0)
- added R0200: 1k, Resistor_SMD:R_0805_2012Metric, F.Cu at (344.8, 32.2)
- added R0201: 1k, Resistor_SMD:R_0805_2012Metric, F.Cu at (344.8, 35.2)
- added R0202: 1k, Resistor_SMD:R_0805_2012Metric, B.Cu at (358.9, 7.67)
- added R0203: 1k, Resistor_SMD:R_0805_2012Metric, B.Cu at (356.6, 7.67)
- added R0204: 10k, Resistor_SMD:R_0805_2012Metric, F.Cu at (344.8, 44.0)
- added R0400: -, Resistor_SMD:R_0805_2012Metric, F.Cu at (125.4, 111.0)
- added R0401: -, Resistor_SMD:R_0805_2012Metric, F.Cu at (125.4, 113.9)
- added R0500: 1k, Resistor_SMD:R_0805_2012Metric, F.Cu at (198.1, 89.9)
- added R0502: 10k, Resistor_SMD:R_0805_2012Metric, F.Cu at (198.1, 92.9)
- added R0503: 10k, Connector_JST:JST_PH_B2B-PH-K_1x02_P2.00mm_Vertical, F.Cu at (198.9, 84.6)
- added R0504: 10k, Resistor_SMD:R_0805_2012Metric, F.Cu at (198.1, 95.8)
- added R0600: 10, Resistor_SMD:R_0805_2012Metric, F.Cu at (120.1, 59.5)
- added R0601: 10, Resistor_SMD:R_0805_2012Metric, F.Cu at (120.1, 62.5)
- added R0602: 10, Resistor_SMD:R_0805_2012Metric, F.Cu at (120.1, 65.4)
- added R0603: 10, Resistor_SMD:R_0805_2012Metric, F.Cu at (120.1, 68.4)
- added R0604: 10, Resistor_SMD:R_0805_2012Metric, F.Cu at (120.1, 71.3)
- added R0605: 10, Resistor_SMD:R_0805_2012Metric, F.Cu at (120.1, 74.3)
- added R0606: 10k, Resistor_SMD:R_0805_2012Metric, F.Cu at (120.1, 77.2)
- added R0607: 10k, Resistor_SMD:R_0805_2012Metric, F.Cu at (124.6, 59.5)
- added R0608: 10k, Resistor_SMD:R_0805_2012Metric, F.Cu at (124.6, 62.5)
- added R0609: 10k, Resistor_SMD:R_0805_2012Metric, F.Cu at (124.6, 65.4)
- added R0610: 10k, Resistor_SMD:R_0805_2012Metric, F.Cu at (124.6, 68.4)
- added R0611: 10k, Resistor_SMD:R_0805_2012Metric, F.Cu at (124.6, 71.3)
- added R0612: 10k, Resistor_SMD:R_0805_2012Metric, F.Cu at (124.6, 74.3)
- added R0613: 10k, Resistor_SMD:R_0805_2012Metric, F.Cu at (124.6, 77.2)
- added R0614: 10k, Resistor_SMD:R_0805_2012Metric, F.Cu at (129.0, 59.5)
- added R0615: 10k, Resistor_SMD:R_0805_2012Metric, F.Cu at (129.0, 62.5)
- added R0616: 10k, Resistor_SMD:R_0805_2012Metric, F.Cu at (129.0, 65.4)
- added R0617: 12.4k, Resistor_SMD:R_0805_2012Metric, F.Cu at (129.0, 68.4)
- added R0618: 51, Resistor_SMD:R_0805_2012Metric, F.Cu at (129.0, 71.3)
- added R0619: 51, Resistor_SMD:R_0805_2012Metric, F.Cu at (129.0, 74.3)
- added R0620: 10, Resistor_SMD:R_0805_2012Metric, F.Cu at (129.0, 77.2)
- added R0621: 82, Resistor_SMD:R_0805_2012Metric, F.Cu at (133.4, 59.5)
- added R0622: 82, Resistor_SMD:R_0805_2012Metric, F.Cu at (133.4, 62.5)
- added R0623: 10k, Resistor_SMD:R_0805_2012Metric, F.Cu at (133.4, 65.4)
- added R0624: 10k, Resistor_SMD:R_0805_2012Metric, F.Cu at (133.4, 68.4)
- added R0625: 10k, Resistor_SMD:R_0805_2012Metric, F.Cu at (133.4, 71.3)
- added R0800: 10, Resistor_SMD:R_0805_2012Metric, F.Cu at (198.1, 101.1)
- added R0801: 10, Resistor_SMD:R_0805_2012Metric, F.Cu at (198.1, 104.1)
- added R0802: 10, Resistor_SMD:R_0805_2012Metric, F.Cu at (198.1, 107.0)
- added R0803: 10, Resistor_SMD:R_0805_2012Metric, F.Cu at (198.1, 110.0)
- added R0900: 10k, Resistor_SMD:R_0805_2012Metric, F.Cu at (317.5, 175.7)
- added R0901: 10k, Resistor_SMD:R_0805_2012Metric, F.Cu at (326.7, 160.6)
- added R0902: 10k, Resistor_SMD:R_0805_2012Metric, F.Cu at (346.4, 174.0)
- added R0903: 10k, Resistor_SMD:R_0805_2012Metric, F.Cu at (312.8, 160.6)
- added R0904: 10k, Resistor_SMD:R_0805_2012Metric, F.Cu at (332.4, 174.0)
- added R0905: 10k, Resistor_SMD:R_0805_2012Metric, F.Cu at (341.0, 161.1)
- added R1000: 22k, Resistor_SMD:R_0805_2012Metric, F.Cu at (140.5, 104.8)
- added R1001: 22k, Resistor_SMD:R_0805_2012Metric, F.Cu at (172.8, 77.7)
- added R1002: 22k, Resistor_SMD:R_0805_2012Metric, F.Cu at (140.5, 77.7)
- added R1003: 22k, Resistor_SMD:R_0805_2012Metric, F.Cu at (183.7, 36.7)
- added R9800: 1k, Resistor_SMD:R_0805_2012Metric, F.Cu at (114.5, 51.9)
- added R9900: 1.2k, Resistor_SMD:R_0805_2012Metric, F.Cu at (168.4, 30.3)
- added R9901: 500, Resistor_SMD:R_0805_2012Metric, F.Cu at (168.4, 33.3)
- added R9902: 10k, Resistor_SMD:R_0805_2012Metric, F.Cu at (168.4, 36.2)
- added R9903: 1.2k, Resistor_SMD:R_0805_2012Metric, F.Cu at (168.4, 39.2)
- added R9904: 500, Resistor_SMD:R_0805_2012Metric, F.Cu at (172.8, 30.3)
- added R9905: 10k, Resistor_SMD:R_0805_2012Metric, F.Cu at (172.8, 33.3)
- added R9906: 3k, Resistor_SMD:R_0805_2012Metric, F.Cu at (172.8, 36.2)
- added R9907: 1k, Resistor_SMD:R_0805_2012Metric, F.Cu at (172.8, 39.2)
- added R9908: 1k, Resistor_SMD:R_0805_2012Metric, F.Cu at (177.2, 30.3)
- added R9909: 1k, Resistor_SMD:R_0805_2012Metric, F.Cu at (177.2, 33.3)
- added R9910: 1k, Resistor_SMD:R_0805_2012Metric, F.Cu at (177.2, 36.2)
- added R9911: 1k, Resistor_SMD:R_0805_2012Metric, F.Cu at (177.2, 39.2)
- added SW0000: Push_Button, Button_Switch_SMD:SW_SPST_PTS647_Sx38, F.Cu at (102.1, 122.8)
- added SWD0: Conn_01x05_Socket, Connector_PinSocket_2.54mm:PinSocket_1x05_P2.54mm_Vertical, F.Cu at (164.7, 146.8)
- added U1: STM32F405RGTx, Package_QFP:LQFP-64_10x10mm_P0.5mm, F.Cu at (114.0, 108.7)
- added U10: RT9193-33GB, Package_TO_SOT_SMD:SOT-23-5, F.Cu at (173.2, 50.1)
- added U2: FT232RL, Package_SO:SSOP-28_5.3x10.2mm_P0.65mm, F.Cu at (359.8, 28.9)
- added U4: W5500, Package_QFP:LQFP-48_7x7mm_P0.5mm, F.Cu at (233.4, 106.5)
- added U5: W25Q32JVSS, Package_SO:SOIC-8_5.3x5.3mm_P1.27mm, F.Cu at (205.5, 103.1)
- added U6: CD4066BPW, Package_SO:TSSOP-14_4.4x5mm_P0.65mm, F.Cu at (116.7, 47.1)
- added U7: LM2596S-ADJ, PCM_Package_TO_SOT_SMD_AKL:TO-263-5_TabPin3_ThermalVias, F.Cu at (147.3, 20.1)
- added U8: LM2596S-ADJ, PCM_Package_TO_SOT_SMD_AKL:TO-263-5_TabPin3_ThermalVias, F.Cu at (147.3, 32.6)
- added U9: LM2596S-ADJ, PCM_Package_TO_SOT_SMD_AKL:TO-263-5_TabPin3_ThermalVias, F.Cu at (147.3, 45.1)
- added USB1: USB_B, Connector_USB:USB_B_OST_USB-B1HSxx_Horizontal, F.Cu at (357.9, 12.9)
- added X0000: 8MHz, Crystal:Crystal_HC49-4H_Vertical, F.Cu at (110.9, 119.2)
- added X0600: 25MHz, Crystal:Crystal_HC49-4H_Vertical, F.Cu at (102.0, 84.7)
Routing:
- net +24V: track 0.00 -> 115.1 mm
- net +5V: track 0.00 -> 107.4 mm
- net Net-(LD0200-K): track 0.00 -> 36.8 mm
- net Net-(LD0201-K): track 0.00 -> 34.9 mm
- net /Motor3/MS3: track 0.00 -> 20.2 mm
- net /Motor1/MS3: track 0.00 -> 19.6 mm
- net /Motor2/MS3: track 0.00 -> 19.5 mm
- net /Motor3/MS1: track 0.00 -> 19.5 mm
- net /Motor0/MS3: track 0.00 -> 19.4 mm
- net /Motor2/A2: track 0.00 -> 19.4 mm
- net /Motor2/B2: track 0.00 -> 19.4 mm
- net /Motor2/B1: track 0.00 -> 19.4 mm
- net /Motor2/A1: track 0.00 -> 19.4 mm
- net /Motor2/MS1: track 0.00 -> 18.8 mm
- net /Motor1/MS1: track 0.00 -> 18.8 mm
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Other:
- board outline added: 109.3 x 56.4 mm
