File: MasterBoard.kicad_pcb (KiCad board)
At the start: 2 copper layers, 109.3 x 56.4 mm, 192 parts, among them J10 WF-2, Q0500 2N7002, SW0000 Push_Button, U1 STM32F405RGTx, U10 RT9193-33GB, U2 FT232RL, U4 W5500, U5 W25Q32JVSS, U6 CD4066BPW, U7 LM2596S-ADJ, U8 LM2596S-ADJ, U9 LM2596S-ADJ, X0000 8MHz, X0600 25MHz

Commit message: Мелкие перестановки, просто кое что прикидывал
Parts:
- removed C0900, C0901, C0902, C0903, C0904, C0905: 10u, Capacitor_SMD:C_0805_2012Metric
- removed C1000, C1002, C1004, C1006: 100u, Capacitor_SMD:CP_Elec_6.3x7.7
- removed C1001, C1003, C1005, C1007: 100u, Capacitor_SMD:C_0805_2012Metric
- removed ES00, ES01, ES02, ES03, ES04, ES05: JST_XH_B3B, Connector_JST:JST_XH_B3B-XH-A_1x03_P2.50mm_Vertical
- removed JP0, JP2, JP4, JP6: SolderJumper_3_Open, Jumper:SolderJumper-3_P1.3mm_Open_RoundedPad1.0x1.5mm
- removed JP1, JP3, JP5, JP7: ~, Connector_PinHeader_2.54mm:PinHeader_1x02_P2.54mm_Vertical
- removed JP1001, JP1002, JP1003, JP1004, JP1005, JP1006, JP1007, JP1008, JP1009, JP1010, JP1011, JP1012: ~, Connector_PinHeader_2.54mm:PinHeader_1x03_P2.54mm_Vertical
- removed M0, M1, M2, M3: ~, Library:MotorSocket
- removed OE0: M3, Connector_JST:JST_XH_B4B-XH-A_1x04_P2.50mm_Vertical
- removed OX0: M0, Connector_JST:JST_XH_B4B-XH-A_1x04_P2.50mm_Vertical
- removed OY0: M1, Connector_JST:JST_XH_B4B-XH-A_1x04_P2.50mm_Vertical
- removed OZ0, OZ1: M2, Connector_JST:JST_XH_B4B-XH-A_1x04_P2.50mm_Vertical
- removed R0900, R0901, R0902, R0903, R0904, R0905: 10k, Resistor_SMD:R_0805_2012Metric
- removed R1000, R1001, R1002, R1003: 22k, Resistor_SMD:R_0805_2012Metric
- removed R9800: 1k, Resistor_SMD:R_0805_2012Metric
- removed U6: CD4066BPW, Package_SO:TSSOP-14_4.4x5mm_P0.65mm
- added C11: 100n, Capacitor_SMD:C_0805_2012Metric, F.Cu at (184.6, 31.3)
- added C12: 100n, Capacitor_SMD:C_0805_2012Metric, F.Cu at (179.5, 35.9)
- added MC1: RJ45_Shielded, Connector_RJ:RJ45_Ninigi_GE, F.Cu at (201.8, 43.5)
- added Q1: MMBT3904, PCM_4ms_Package_SOT:SOT-23, F.Cu at (188.2, 46.0)
- added Q2: MMBT3904, PCM_4ms_Package_SOT:SOT-23, F.Cu at (192.8, 46.0)
- added Q3: MMBT3904, PCM_4ms_Package_SOT:SOT-23, F.Cu at (188.2, 39.5)
- added Q4: MMBT3904, PCM_4ms_Package_SOT:SOT-23, F.Cu at (192.8, 39.5)
- added R626: 10k, Resistor_SMD:R_0805_2012Metric, F.Cu at (189.9, 43.2)
- added R627: 10k, Resistor_SMD:R_0805_2012Metric, F.Cu at (195.8, 45.1)
- added R628: 10k, Resistor_SMD:R_0805_2012Metric, F.Cu at (184.6, 47.0)
- added R629: 10k, Resistor_SMD:R_0805_2012Metric, F.Cu at (184.6, 40.4)
- added R630: 10k, Resistor_SMD:R_0805_2012Metric, F.Cu at (189.9, 36.9)
- added R631: 10k, Resistor_SMD:R_0805_2012Metric, F.Cu at (195.8, 38.6)
- added R632: 10k, Resistor_SMD:R_0805_2012Metric, F.Cu at (187.1, 29.4)
- added R633: 10k, Resistor_SMD:R_0805_2012Metric, F.Cu at (192.2, 30.4)
- added R634: 15k, Resistor_SMD:R_0805_2012Metric, F.Cu at (189.3, 31.2)
- added R635: 10k, Resistor_SMD:R_0805_2012Metric, F.Cu at (181.8, 34.1)
- added R636: 15k, Resistor_SMD:R_0805_2012Metric, F.Cu at (184.0, 35.9)
- added R637: 10k, Resistor_SMD:R_0805_2012Metric, F.Cu at (186.8, 35.0)
- D0200, R0202, R0203: moved to F.Cu
- moved ETH0 309.1 mm to (37.8, 73.4), turned to 0 degrees
- moved C0200 266.8 mm to (118.8, 81.0)
- moved C0201 266.8 mm to (118.8, 84.0)
- moved C0202 266.8 mm to (118.8, 87.0)
- moved C0203 266.8 mm to (118.8, 90.0)
- moved USB1 255.3 mm to (108.9, 69.4)
- moved U2 254.9 mm to (111.3, 85.5), turned to 0 degrees
- moved LD0200 253.7 mm to (123.3, 81.0), turned to 0 degrees
- moved LD0201 252.6 mm to (123.3, 84.0), turned to 0 degrees
- moved D0200 246.0 mm to (123.2, 87.0)
- moved R0202 239.8 mm to (127.1, 69.2), turned to 0 degrees
- moved R0203 238.3 mm to (127.1, 72.2), turned to 0 degrees
- moved R0200 219.9 mm to (127.1, 63.3)
- moved R0201 219.9 mm to (127.1, 66.3)
- moved R0204 219.9 mm to (127.1, 75.1)
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Connections:
- U1 pad 22: /X0_ES -> /STM32F405RG/PA6
- U1 pad 23: /Y0_ES -> /STM32F405RG/PA7
- U1 pad 25: /M0_DIR -> /STM32F405RG/PC5
- U1 pad 26: /Y1_ES -> /STM32F405RG/PB0
- U1 pad 27: /Z1_ES -> /STM32F405RG/PB1
- U1 pad 28: /M0_SW -> /STM32F405RG/PB2
- U1 pad 37: /M1_DIR -> /STM32F405RG/PC6
- U1 pad 38: /M2_DIR -> /STM32F405RG/PC7
- U1 pad 39: /M3_DIR -> /STM32F405RG/PC8
- U1 pad 40: /M3_SW -> /STM32F405RG/PC9
- U1 pad 41: /M0_STEP -> /STM32F405RG/PA8
- U1 pad 42: /M1_STEP -> /STM32F405RG/PA9
- U1 pad 43: /M2_STEP -> /STM32F405RG/PA10
- U1 pad 44: /M3_STEP -> /STM32F405RG/PA11
- U1 pad 45: /Z0_ES -> /STM32F405RG/PA12
- U1 pad 50: /X1_ES -> /STM32F405RG/PA15
- U1 pad 56: /M1_SW -> /STM32F405RG/PB4
- U1 pad 57: /M2_SW -> /STM32F405RG/PB5
- U1 pad 59: /M_UART -> /M_UART_RX
Routing:
- net +24V: track 115.1 -> 0.00 mm
- net +5V: track 107.4 -> 0.00 mm
- net Net-(LD0200-K): track 36.8 -> 0.00 mm
- net Net-(LD0201-K): track 34.9 -> 0.00 mm
- net /Motor3/MS3: track 20.2 -> 0.00 mm
- net /Motor1/MS3: track 19.6 -> 0.00 mm
- net /Motor2/MS3: track 19.5 -> 0.00 mm
- net /Motor3/MS1: track 19.5 -> 0.00 mm
- net /Motor0/MS3: track 19.4 -> 0.00 mm
- net /Motor2/A2: track 19.4 -> 0.00 mm
- net /Motor2/B2: track 19.4 -> 0.00 mm
- net /Motor2/B1: track 19.4 -> 0.00 mm
- net /Motor2/A1: track 19.4 -> 0.00 mm
- net /Motor2/MS1: track 18.8 -> 0.00 mm
- net /Motor1/MS1: track 18.8 -> 0.00 mm
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Other:
- board outline removed

Commit message: Начал трассировать плату
Parts:
- removed C0000, C0003, C0004, C0005, C0006, C0007, C0200, C0203, C0500, C0602, C0603, C0606, C9910, C9913: 100n, Capacitor_SMD:C_0805_2012Metric
- removed C0001, C0002: 2.2u, Capacitor_SMD:C_0805_2012Metric
- removed C0008, C9909: 1u, Capacitor_SMD:C_0805_2012Metric
- removed C0009, C0010: 20p, Capacitor_SMD:C_0805_2012Metric
- removed C0201, C0601: 4.7u, Capacitor_SMD:C_0805_2012Metric
- removed C0202, C0800, C9912: 10u, Capacitor_SMD:C_0805_2012Metric
- removed C0600, C0609, C9902, C9905, C9908: 10n, Capacitor_SMD:C_0805_2012Metric
- removed C0604, C0605: 18p, Capacitor_SMD:C_0805_2012Metric
- removed C0607, C9911: 22n, Capacitor_SMD:C_0805_2012Metric
- removed C0608, C0610: 6.8n, Capacitor_SMD:C_0805_2012Metric
- removed C9900, C9903, C9906: 100u, Capacitor_SMD:C_0805_2012Metric
- removed C9901, C9904, C9907: 220u, Capacitor_SMD:C_0805_2012Metric
- removed D0200, D9800: BAT60A, Diode_SMD:D_SOD-323
- removed D9900, D9901, D9902: 1N5822, PCM_4ms_Diode:D_DO-214AC_SMA
- removed DISP0: IDC-14, Connector_IDC:IDC-Header_2x07_P2.54mm_Vertical
- removed ETH0: RJ45_Hanrun_HR911105A_Horizontal, Connector_RJ:RJ45_Hanrun_HR911105A_Horizontal
- removed FAN0: Fan_CPU_4pin, Connector:FanPinHeader_1x04_P2.54mm_Vertical
- removed HOTEND0: IDC-16, Connector_IDC:IDC-Header_2x08_P2.54mm_Vertical
- removed J10: WF-2, Library:WF-2
- removed L9900, L9901, L9902: 33u, Inductor_SMD:L_APV_APH0650
- removed LD0200, LD0201, LD0500, LD9900, LD9901, LD9902, LD9903: ~, LED_SMD:LED_0805_2012Metric
- removed PWR0: Conn_01x02, Library:KLS2
- removed Q0500: 2N7002, PCM_4ms_Package_SOT:SOT-23
- removed R0000: 100k, Resistor_SMD:R_0805_2012Metric
- removed R0200, R0201, R0202, R0203, R0500, R9907, R9908, R9909, R9910, R9911: 1k, Resistor_SMD:R_0805_2012Metric
- removed R0204, R0502, R0504, R0606, R0607, R0608, R0609, R0610, R0611, R0612, R0613, R0614, R0615, R0616, R0623, R0624, R0625, R626, R627, R628, R629, R630, R631, R632, R633, R635, R637, R9902, R9905: 10k, Resistor_SMD:R_0805_2012Metric
- removed R0400, R0401: -, Resistor_SMD:R_0805_2012Metric
- removed R0503: 10k, Connector_JST:JST_PH_B2B-PH-K_1x02_P2.00mm_Vertical
- removed R0600, R0601, R0602, R0603, R0604, R0605, R0620, R0800, R0801, R0802, R0803: 10, Resistor_SMD:R_0805_2012Metric
- removed R0617: 12.4k, Resistor_SMD:R_0805_2012Metric
- removed R0618, R0619: 51, Resistor_SMD:R_0805_2012Metric
- removed R0621, R0622: 82, Resistor_SMD:R_0805_2012Metric
- removed R634, R636: 15k, Resistor_SMD:R_0805_2012Metric
- removed R9900, R9903: 1.2k, Resistor_SMD:R_0805_2012Metric
- removed R9901, R9904: 500, Resistor_SMD:R_0805_2012Metric
- removed R9906: 3k, Resistor_SMD:R_0805_2012Metric
- removed SW0000: Push_Button, Button_Switch_SMD:SW_SPST_PTS647_Sx38
- removed SWD0: Conn_01x05_Socket, Connector_PinSocket_2.54mm:PinSocket_1x05_P2.54mm_Vertical
- removed U10: RT9193-33GB, Package_TO_SOT_SMD:SOT-23-5
- removed U7, U8, U9: LM2596S-ADJ, PCM_Package_TO_SOT_SMD_AKL:TO-263-5_TabPin3_ThermalVias
- removed X0000: 8MHz, Crystal:Crystal_HC49-4H_Vertical
- removed X0600: 25MHz, Crystal:Crystal_HC49-4H_Vertical
- added C1: 100u, Capacitor_SMD:C_0805_2012Metric, F.Cu at (63.1, 19.8)
- added C10: 1u, Capacitor_SMD:C_0805_2012Metric, F.Cu at (67.5, 31.9)
- added C13: 10u, Capacitor_SMD:C_0805_2012Metric, F.Cu at (72.0, 25.8)
- added C14: 100n, Capacitor_SMD:C_0805_2012Metric, F.Cu at (72.0, 28.8)
- added C15: 100n, Capacitor_SMD:C_0805_2012Metric, F.Cu at (35.2, 79.3)
- added C16: 2.2u, Capacitor_SMD:C_0805_2012Metric, F.Cu at (35.2, 82.3)
- added C17: 2.2u, Capacitor_SMD:C_0805_2012Metric, F.Cu at (35.2, 85.3)
- added C18: 100n, Capacitor_SMD:C_0805_2012Metric, F.Cu at (35.2, 88.3)
- added C19: 100n, Capacitor_SMD:C_0805_2012Metric, F.Cu at (35.2, 91.3)
- added C2: 100u, Capacitor_SMD:C_0805_2012Metric, F.Cu at (63.1, 22.8)
- added C20: 100n, Capacitor_SMD:C_0805_2012Metric, F.Cu at (39.7, 79.3)
- added C21: 20p, Capacitor_SMD:C_0805_2012Metric, F.Cu at (39.7, 82.3)
- added C22: 20p, Capacitor_SMD:C_0805_2012Metric, F.Cu at (39.7, 85.3)
- added C23: 100n, Capacitor_SMD:C_0805_2012Metric, F.Cu at (39.7, 88.3)
- added C24: 100n, Capacitor_SMD:C_0805_2012Metric, F.Cu at (39.7, 91.3)
- added C25: 100n, Capacitor_SMD:C_0805_2012Metric, F.Cu at (44.1, 79.3)
- added C26: 100n, Capacitor_SMD:C_0805_2012Metric, F.Cu at (44.1, 82.3)
- added C27: 100n, Capacitor_SMD:C_0805_2012Metric, F.Cu at (44.1, 85.3)
- added C28: 4.7u, Capacitor_SMD:C_0805_2012Metric, F.Cu at (44.1, 88.3)
- added C29: 10u, Capacitor_SMD:C_0805_2012Metric, F.Cu at (155.1, 138.7)
- added C3: 100u, Capacitor_SMD:C_0805_2012Metric, F.Cu at (63.1, 25.8)
- added C30: 100n, Capacitor_SMD:C_0805_2012Metric, F.Cu at (155.1, 141.7)
- added C31: 4.7u, Capacitor_SMD:C_0805_2012Metric, F.Cu at (155.1, 144.7)
- added C32: 100n, Capacitor_SMD:C_0805_2012Metric, F.Cu at (155.1, 147.7)
- added C33: 100n, Capacitor_SMD:C_0805_2012Metric, F.Cu at (152.5, 107.3)
- added C34: 100n, Capacitor_SMD:C_0805_2012Metric, F.Cu at (152.5, 110.4)
- added C35: 100n, Capacitor_SMD:C_0805_2012Metric, F.Cu at (152.5, 113.4)
- added C36: 100n, Capacitor_SMD:C_0805_2012Metric, F.Cu at (285.4, 236.1)
- added C37: 100n, Capacitor_SMD:C_0805_2012Metric, F.Cu at (285.4, 239.1)
- added C38: 100n, Capacitor_SMD:C_0805_2012Metric, F.Cu at (99.0, 136.4)
- added C39: 100n, Capacitor_SMD:C_0805_2012Metric, F.Cu at (99.0, 139.4)
- added C4: 220u, Capacitor_SMD:C_0805_2012Metric, F.Cu at (63.1, 28.8)
- added C40: 100n, Capacitor_SMD:C_0805_2012Metric, F.Cu at (165.1, 67.4)
- added C41: 100n, Capacitor_SMD:C_0805_2012Metric, F.Cu at (165.1, 70.4)
- added C42: 100n, Capacitor_SMD:C_0805_2012Metric, F.Cu at (132.1, 32.9)
- added C43: 100n, Capacitor_SMD:C_0805_2012Metric, F.Cu at (132.1, 35.9)
- added C44: 100n, Capacitor_SMD:C_0805_2012Metric, F.Cu at (99.0, 101.9)
- added C45: 100n, Capacitor_SMD:C_0805_2012Metric, F.Cu at (99.0, 104.9)
- added C46: 100n, Capacitor_SMD:C_0805_2012Metric, F.Cu at (132.1, 67.4)
- added C47: 100n, Capacitor_SMD:C_0805_2012Metric, F.Cu at (132.1, 70.4)
- added C48: 100n, Capacitor_SMD:C_0805_2012Metric, F.Cu at (132.1, 101.9)
- added C49: 100n, Capacitor_SMD:C_0805_2012Metric, F.Cu at (132.1, 104.9)
- added C5: 220u, Capacitor_SMD:C_0805_2012Metric, F.Cu at (63.1, 31.9)
- added C50: 100n, Capacitor_SMD:C_0805_2012Metric, F.Cu at (99.0, 67.4)
- added C51: 100n, Capacitor_SMD:C_0805_2012Metric, F.Cu at (99.0, 70.4)
- added C52: 100n, Capacitor_SMD:C_0805_2012Metric, F.Cu at (165.1, 32.9)
- added C53: 100n, Capacitor_SMD:C_0805_2012Metric, F.Cu at (165.1, 35.9)
- added C54: 100n, Capacitor_SMD:C_0805_2012Metric, F.Cu at (99.0, 32.9)
- added C55: 100n, Capacitor_SMD:C_0805_2012Metric, F.Cu at (99.0, 35.9)
- added C6: 220u, Capacitor_SMD:C_0805_2012Metric, F.Cu at (67.5, 19.8)
- added C7: 10n, Capacitor_SMD:C_0805_2012Metric, F.Cu at (67.5, 22.8)
- added C8: 10n, Capacitor_SMD:C_0805_2012Metric, F.Cu at (67.5, 25.8)
- added C9: 10n, Capacitor_SMD:C_0805_2012Metric, F.Cu at (67.5, 28.8)
- added D1: BAT60A, Diode_SMD:D_SOD-323, F.Cu at (47.0, 122.5)
- added D2: 1N5822, PCM_4ms_Diode:D_DO-214AC_SMA, F.Cu at (54.4, 45.2)
- added D3: 1N5822, PCM_4ms_Diode:D_DO-214AC_SMA, F.Cu at (54.4, 49.6)
- added D4: 1N5822, PCM_4ms_Diode:D_DO-214AC_SMA, F.Cu at (54.4, 53.9)
- added D5: BAT60A, Diode_SMD:D_SOD-323, F.Cu at (159.4, 144.8)
- added ESA1: ESA, Connector_JST:JST_PH_B3B-PH-K_1x03_P2.00mm_Vertical, F.Cu at (286.2, 224.2)
- added ESA10: ESA, Connector_JST:JST_PH_B3B-PH-K_1x03_P2.00mm_Vertical, F.Cu at (99.8, 21.0)
- added ESA2: ESA, Connector_JST:JST_PH_B3B-PH-K_1x03_P2.00mm_Vertical, F.Cu at (99.8, 124.5)
- added ESA3: ESA, Connector_JST:JST_PH_B3B-PH-K_1x03_P2.00mm_Vertical, F.Cu at (165.9, 55.5)
- added ESA4: ESA, Connector_JST:JST_PH_B3B-PH-K_1x03_P2.00mm_Vertical, F.Cu at (132.8, 21.0)
- added ESA5: ESA, Connector_JST:JST_PH_B3B-PH-K_1x03_P2.00mm_Vertical, F.Cu at (99.8, 90.0)
- added ESA6: ESA, Connector_JST:JST_PH_B3B-PH-K_1x03_P2.00mm_Vertical, F.Cu at (132.8, 55.5)
- added ESA7: ESA, Connector_JST:JST_PH_B3B-PH-K_1x03_P2.00mm_Vertical, F.Cu at (132.8, 90.0)
- added ESA8: ESA, Connector_JST:JST_PH_B3B-PH-K_1x03_P2.00mm_Vertical, F.Cu at (99.8, 55.5)
- added ESA9: ESA, Connector_JST:JST_PH_B3B-PH-K_1x03_P2.00mm_Vertical, F.Cu at (165.9, 21.0)
- added ESB1: ESB, Connector_JST:JST_PH_B3B-PH-K_1x03_P2.00mm_Vertical, F.Cu at (286.2, 230.8)
- added ESB10: ESB, Connector_JST:JST_PH_B3B-PH-K_1x03_P2.00mm_Vertical, F.Cu at (99.8, 27.6)
- added ESB2: ESB, Connector_JST:JST_PH_B3B-PH-K_1x03_P2.00mm_Vertical, F.Cu at (99.8, 131.1)
- added ESB3: ESB, Connector_JST:JST_PH_B3B-PH-K_1x03_P2.00mm_Vertical, F.Cu at (165.9, 62.1)
- added ESB4: ESB, Connector_JST:JST_PH_B3B-PH-K_1x03_P2.00mm_Vertical, F.Cu at (132.8, 27.6)
- added ESB5: ESB, Connector_JST:JST_PH_B3B-PH-K_1x03_P2.00mm_Vertical, F.Cu at (99.8, 96.6)
- added ESB6: ESB, Connector_JST:JST_PH_B3B-PH-K_1x03_P2.00mm_Vertical, F.Cu at (132.8, 62.1)
- added ESB7: ESB, Connector_JST:JST_PH_B3B-PH-K_1x03_P2.00mm_Vertical, F.Cu at (132.8, 96.6)
- added ESB8: ESB, Connector_JST:JST_PH_B3B-PH-K_1x03_P2.00mm_Vertical, F.Cu at (99.8, 62.1)
- added ESB9: ESB, Connector_JST:JST_PH_B3B-PH-K_1x03_P2.00mm_Vertical, F.Cu at (165.9, 27.6)
- added FAN1: Fan_CPU_4pin, Connector:FanPinHeader_1x04_P2.54mm_Vertical, F.Cu at (159.4, 113.3)
- added J1: HX711, Connector_JST:JST_PH_B4B-PH-K_1x04_P2.00mm_Vertical, F.Cu at (43.2, 97.6)
- added J2: HX711, Connector_JST:JST_PH_B4B-PH-K_1x04_P2.00mm_Vertical, F.Cu at (43.2, 104.1)
- added J3: HX711, Connector_JST:JST_PH_B4B-PH-K_1x04_P2.00mm_Vertical, F.Cu at (43.2, 110.7)
- added J4: HX711, Connector_JST:JST_PH_B4B-PH-K_1x04_P2.00mm_Vertical, F.Cu at (43.2, 117.2)
- added J5: WF-2, Library:WF-2, F.Cu at (154.0, 90.4)
- added J6: WF-2, Library:WF-2, F.Cu at (154.0, 96.6)
- added J7: WF-2, Library:WF-2, F.Cu at (154.0, 102.8)
- added L1: 33u, Inductor_SMD:L_APV_APH0650, F.Cu at (55.9, 22.4)
- added L2: 33u, Inductor_SMD:L_APV_APH0650, F.Cu at (55.9, 30.7)
- added L3: 33u, Inductor_SMD:L_APV_APH0650, F.Cu at (55.9, 38.9)
- added LD1: ~, LED_SMD:LED_0805_2012Metric, F.Cu at (63.1, 46.7)
- added LD10: ~, LED_SMD:LED_0805_2012Metric, F.Cu at (168.2, 94.9)
- added LD2: ~, LED_SMD:LED_0805_2012Metric, F.Cu at (63.1, 49.7)
- added LD3: ~, LED_SMD:LED_0805_2012Metric, F.Cu at (63.1, 52.8)
- added LD4: ~, LED_SMD:LED_0805_2012Metric, F.Cu at (63.1, 55.8)
- added LD5: ~, LED_SMD:LED_0805_2012Metric, F.Cu at (48.6, 90.5)
- added LD6: ~, LED_SMD:LED_0805_2012Metric, F.Cu at (159.5, 138.7)
- added LD7: ~, LED_SMD:LED_0805_2012Metric, F.Cu at (159.5, 141.8)
- added LD8: ~, LED_SMD:LED_0805_2012Metric, F.Cu at (168.2, 88.8)
- added LD9: ~, LED_SMD:LED_0805_2012Metric, F.Cu at (168.2, 91.9)
- added MC10: RJ45_Shielded, Connector_RJ:RJ45_Ninigi_GE, F.Cu at (82.1, 23.5)
- added MC2: RJ45_Shielded, Connector_RJ:RJ45_Ninigi_GE, F.Cu at (82.1, 127.0)
- added MC3: RJ45_Shielded, Connector_RJ:RJ45_Ninigi_GE, F.Cu at (148.1, 58.0)
- added MC4: RJ45_Shielded, Connector_RJ:RJ45_Ninigi_GE, F.Cu at (115.1, 23.5)
- added MC5: RJ45_Shielded, Connector_RJ:RJ45_Ninigi_GE, F.Cu at (82.1, 92.5)
- added MC6: RJ45_Shielded, Connector_RJ:RJ45_Ninigi_GE, F.Cu at (115.1, 58.0)
- added MC7: RJ45_Shielded, Connector_RJ:RJ45_Ninigi_GE, F.Cu at (115.1, 92.5)
- added MC8: RJ45_Shielded, Connector_RJ:RJ45_Ninigi_GE, F.Cu at (82.1, 58.0)
- added MC9: RJ45_Shielded, Connector_RJ:RJ45_Ninigi_GE, F.Cu at (148.1, 23.5)
- added PWR1: Conn_01x02, Library:KLS2, F.Cu at (69.2, 48.7)
- added Q10: MMBT3904, PCM_4ms_Package_SOT:SOT-23, F.Cu at (78.4, 144.8)
- added Q11: MMBT3904, PCM_4ms_Package_SOT:SOT-23, F.Cu at (82.9, 144.8)
- added Q12: MMBT3904, PCM_4ms_Package_SOT:SOT-23, F.Cu at (87.3, 144.8)
- added Q13: MMBT3904, PCM_4ms_Package_SOT:SOT-23, F.Cu at (91.8, 144.8)
- added Q14: MMBT3904, PCM_4ms_Package_SOT:SOT-23, F.Cu at (144.5, 75.8)
- added Q15: MMBT3904, PCM_4ms_Package_SOT:SOT-23, F.Cu at (149.0, 75.8)
- added Q16: MMBT3904, PCM_4ms_Package_SOT:SOT-23, F.Cu at (153.4, 75.8)
- added Q17: MMBT3904, PCM_4ms_Package_SOT:SOT-23, F.Cu at (157.9, 75.8)
- added Q18: MMBT3904, PCM_4ms_Package_SOT:SOT-23, F.Cu at (111.5, 41.3)
- added Q19: MMBT3904, PCM_4ms_Package_SOT:SOT-23, F.Cu at (115.9, 41.3)
- added Q20: MMBT3904, PCM_4ms_Package_SOT:SOT-23, F.Cu at (120.4, 41.3)
- added Q21: MMBT3904, PCM_4ms_Package_SOT:SOT-23, F.Cu at (124.8, 41.3)
- added Q22: MMBT3904, PCM_4ms_Package_SOT:SOT-23, F.Cu at (78.4, 110.3)
- added Q23: MMBT3904, PCM_4ms_Package_SOT:SOT-23, F.Cu at (82.9, 110.3)
- added Q24: MMBT3904, PCM_4ms_Package_SOT:SOT-23, F.Cu at (87.3, 110.3)
- added Q25: MMBT3904, PCM_4ms_Package_SOT:SOT-23, F.Cu at (91.8, 110.3)
- added Q26: MMBT3904, PCM_4ms_Package_SOT:SOT-23, F.Cu at (111.5, 75.8)
- added Q27: MMBT3904, PCM_4ms_Package_SOT:SOT-23, F.Cu at (115.9, 75.8)
- added Q28: MMBT3904, PCM_4ms_Package_SOT:SOT-23, F.Cu at (120.4, 75.8)
- added Q29: MMBT3904, PCM_4ms_Package_SOT:SOT-23, F.Cu at (124.8, 75.8)
- added Q30: MMBT3904, PCM_4ms_Package_SOT:SOT-23, F.Cu at (111.5, 110.3)
- added Q31: MMBT3904, PCM_4ms_Package_SOT:SOT-23, F.Cu at (115.9, 110.3)
- added Q32: MMBT3904, PCM_4ms_Package_SOT:SOT-23, F.Cu at (120.4, 110.3)
- added Q33: MMBT3904, PCM_4ms_Package_SOT:SOT-23, F.Cu at (124.8, 110.3)
- added Q34: MMBT3904, PCM_4ms_Package_SOT:SOT-23, F.Cu at (78.4, 75.8)
- added Q35: MMBT3904, PCM_4ms_Package_SOT:SOT-23, F.Cu at (82.9, 75.8)
- added Q36: MMBT3904, PCM_4ms_Package_SOT:SOT-23, F.Cu at (87.3, 75.8)
- added Q37: MMBT3904, PCM_4ms_Package_SOT:SOT-23, F.Cu at (91.8, 75.8)
- added Q38: MMBT3904, PCM_4ms_Package_SOT:SOT-23, F.Cu at (144.5, 41.3)
- added Q39: MMBT3904, PCM_4ms_Package_SOT:SOT-23, F.Cu at (149.0, 41.3)
- added Q40: MMBT3904, PCM_4ms_Package_SOT:SOT-23, F.Cu at (153.4, 41.3)
- added Q41: MMBT3904, PCM_4ms_Package_SOT:SOT-23, F.Cu at (157.9, 41.3)
- added Q42: MMBT3904, PCM_4ms_Package_SOT:SOT-23, F.Cu at (78.4, 41.3)
- added Q43: MMBT3904, PCM_4ms_Package_SOT:SOT-23, F.Cu at (82.9, 41.3)
- added Q44: MMBT3904, PCM_4ms_Package_SOT:SOT-23, F.Cu at (87.3, 41.3)
- added Q45: MMBT3904, PCM_4ms_Package_SOT:SOT-23, F.Cu at (91.8, 41.3)
- added Q5: 2N7002, PCM_4ms_Package_SOT:SOT-23, F.Cu at (168.3, 107.3)
- added Q6: MMBT3904, PCM_4ms_Package_SOT:SOT-23, F.Cu at (264.8, 244.5)
- added Q7: MMBT3904, PCM_4ms_Package_SOT:SOT-23, F.Cu at (269.3, 244.5)
- added Q8: MMBT3904, PCM_4ms_Package_SOT:SOT-23, F.Cu at (273.7, 244.5)
- added Q9: MMBT3904, PCM_4ms_Package_SOT:SOT-23, F.Cu at (278.2, 244.5)
- added R1: 1.2k, Resistor_SMD:R_0805_2012Metric, F.Cu at (63.1, 34.8)
- added R10: 1k, Resistor_SMD:R_0805_2012Metric, F.Cu at (71.9, 37.8)
- added R100: 10k, Resistor_SMD:R_0805_2012Metric, F.Cu at (100.6, 112.4)
- added R101: 10k, Resistor_SMD:R_0805_2012Metric, F.Cu at (100.6, 115.4)
- added R102: 10k, Resistor_SMD:R_0805_2012Metric, F.Cu at (100.6, 118.3)
- added R103: 10k, Resistor_SMD:R_0805_2012Metric, F.Cu at (105.0, 109.5)
- added R104: 10k, Resistor_SMD:R_0805_2012Metric, F.Cu at (105.0, 112.4)
- added R105: 10k, Resistor_SMD:R_0805_2012Metric, F.Cu at (105.0, 115.4)
- added R106: 10k, Resistor_SMD:R_0805_2012Metric, F.Cu at (105.0, 118.3)
- added R107: 10k, Resistor_SMD:R_0805_2012Metric, F.Cu at (129.3, 75.0)
- added R108: 10k, Resistor_SMD:R_0805_2012Metric, F.Cu at (129.3, 77.9)
- added R109: 15k, Resistor_SMD:R_0805_2012Metric, F.Cu at (129.3, 80.9)
- added R11: 1k, Resistor_SMD:R_0805_2012Metric, F.Cu at (71.9, 40.7)
- added R110: 15k, Resistor_SMD:R_0805_2012Metric, F.Cu at (129.3, 83.8)
- added R111: 10k, Resistor_SMD:R_0805_2012Metric, F.Cu at (133.7, 75.0)
- added R112: 10k, Resistor_SMD:R_0805_2012Metric, F.Cu at (133.7, 77.9)
- added R113: 10k, Resistor_SMD:R_0805_2012Metric, F.Cu at (133.7, 80.9)
- added R114: 10k, Resistor_SMD:R_0805_2012Metric, F.Cu at (133.7, 83.8)
- added R115: 10k, Resistor_SMD:R_0805_2012Metric, F.Cu at (138.1, 75.0)
- added R116: 10k, Resistor_SMD:R_0805_2012Metric, F.Cu at (138.1, 77.9)
- added R117: 10k, Resistor_SMD:R_0805_2012Metric, F.Cu at (138.1, 80.9)
- added R118: 10k, Resistor_SMD:R_0805_2012Metric, F.Cu at (138.1, 83.8)
- added R119: 10k, Resistor_SMD:R_0805_2012Metric, F.Cu at (129.3, 109.5)
- added R12: 1k, Resistor_SMD:R_0805_2012Metric, F.Cu at (71.9, 43.7)
- added R120: 10k, Resistor_SMD:R_0805_2012Metric, F.Cu at (129.3, 112.4)
- added R121: 15k, Resistor_SMD:R_0805_2012Metric, F.Cu at (129.3, 115.4)
- added R122: 15k, Resistor_SMD:R_0805_2012Metric, F.Cu at (129.3, 118.3)
- added R123: 10k, Resistor_SMD:R_0805_2012Metric, F.Cu at (133.7, 109.5)
- added R124: 10k, Resistor_SMD:R_0805_2012Metric, F.Cu at (133.7, 112.4)
- added R125: 10k, Resistor_SMD:R_0805_2012Metric, F.Cu at (133.7, 115.4)
- added R126: 10k, Resistor_SMD:R_0805_2012Metric, F.Cu at (133.7, 118.3)
- added R127: 10k, Resistor_SMD:R_0805_2012Metric, F.Cu at (138.1, 109.5)
- added R128: 10k, Resistor_SMD:R_0805_2012Metric, F.Cu at (138.1, 112.4)
- added R129: 10k, Resistor_SMD:R_0805_2012Metric, F.Cu at (138.1, 115.4)
- added R13: 10k, Resistor_SMD:R_0805_2012Metric, F.Cu at (53.7, 60.8)
- added R130: 10k, Resistor_SMD:R_0805_2012Metric, F.Cu at (138.1, 118.3)
- added R131: 10k, Resistor_SMD:R_0805_2012Metric, F.Cu at (96.2, 75.0)
- added R132: 10k, Resistor_SMD:R_0805_2012Metric, F.Cu at (96.2, 77.9)
- added R133: 15k, Resistor_SMD:R_0805_2012Metric, F.Cu at (96.2, 80.9)
- added R134: 15k, Resistor_SMD:R_0805_2012Metric, F.Cu at (96.2, 83.8)
- added R135: 10k, Resistor_SMD:R_0805_2012Metric, F.Cu at (100.6, 75.0)
- added R136: 10k, Resistor_SMD:R_0805_2012Metric, F.Cu at (100.6, 77.9)
- added R137: 10k, Resistor_SMD:R_0805_2012Metric, F.Cu at (100.6, 80.9)
- added R138: 10k, Resistor_SMD:R_0805_2012Metric, F.Cu at (100.6, 83.8)
- added R139: 10k, Resistor_SMD:R_0805_2012Metric, F.Cu at (105.0, 75.0)
- added R14: 10, Resistor_SMD:R_0805_2012Metric, F.Cu at (53.7, 63.7)
- added R140: 10k, Resistor_SMD:R_0805_2012Metric, F.Cu at (105.0, 77.9)
- added R141: 10k, Resistor_SMD:R_0805_2012Metric, F.Cu at (105.0, 80.9)
- added R142: 10k, Resistor_SMD:R_0805_2012Metric, F.Cu at (105.0, 83.8)
- added R143: 10k, Resistor_SMD:R_0805_2012Metric, F.Cu at (162.3, 40.5)
- added R144: 10k, Resistor_SMD:R_0805_2012Metric, F.Cu at (162.3, 43.4)
- added R145: 15k, Resistor_SMD:R_0805_2012Metric, F.Cu at (162.3, 46.4)
- added R146: 15k, Resistor_SMD:R_0805_2012Metric, F.Cu at (162.3, 49.3)
- added R147: 10k, Resistor_SMD:R_0805_2012Metric, F.Cu at (166.7, 40.5)
- added R148: 10k, Resistor_SMD:R_0805_2012Metric, F.Cu at (166.7, 43.4)
- added R149: 10k, Resistor_SMD:R_0805_2012Metric, F.Cu at (166.7, 46.4)
- added R15: 10, Resistor_SMD:R_0805_2012Metric, F.Cu at (53.7, 66.7)
- added R150: 10k, Resistor_SMD:R_0805_2012Metric, F.Cu at (166.7, 49.3)
- added R151: 10k, Resistor_SMD:R_0805_2012Metric, F.Cu at (171.1, 40.5)
- added R152: 10k, Resistor_SMD:R_0805_2012Metric, F.Cu at (171.1, 43.4)
- added R153: 10k, Resistor_SMD:R_0805_2012Metric, F.Cu at (171.1, 46.4)
- added R154: 10k, Resistor_SMD:R_0805_2012Metric, F.Cu at (171.1, 49.3)
- added R155: 10k, Resistor_SMD:R_0805_2012Metric, F.Cu at (96.2, 40.5)
- added R156: 10k, Resistor_SMD:R_0805_2012Metric, F.Cu at (96.2, 43.4)
- added R157: 15k, Resistor_SMD:R_0805_2012Metric, F.Cu at (96.2, 46.4)
- added R158: 15k, Resistor_SMD:R_0805_2012Metric, F.Cu at (96.2, 49.3)
- added R159: 10k, Resistor_SMD:R_0805_2012Metric, F.Cu at (100.6, 40.5)
- added R16: 10k, Resistor_SMD:R_0805_2012Metric, F.Cu at (53.7, 69.6)
- added R160: 10k, Resistor_SMD:R_0805_2012Metric, F.Cu at (100.6, 43.4)
- added R161: 10k, Resistor_SMD:R_0805_2012Metric, F.Cu at (100.6, 46.4)
- added R162: 10k, Resistor_SMD:R_0805_2012Metric, F.Cu at (100.6, 49.3)
- added R163: 10k, Resistor_SMD:R_0805_2012Metric, F.Cu at (105.0, 40.5)
- added R164: 10k, Resistor_SMD:R_0805_2012Metric, F.Cu at (105.0, 43.4)
- added R165: 10k, Resistor_SMD:R_0805_2012Metric, F.Cu at (105.0, 46.4)
- added R166: 10k, Resistor_SMD:R_0805_2012Metric, F.Cu at (105.0, 49.3)
- added R17: 10, Resistor_SMD:R_0805_2012Metric, F.Cu at (53.7, 72.6)
- added R18: 10, Resistor_SMD:R_0805_2012Metric, F.Cu at (53.7, 75.5)
- added R19: 10, Resistor_SMD:R_0805_2012Metric, F.Cu at (58.1, 60.8)
- added R2: 1.2k, Resistor_SMD:R_0805_2012Metric, F.Cu at (63.1, 37.8)
- added R20: 10, Resistor_SMD:R_0805_2012Metric, F.Cu at (58.1, 63.7)
- added R21: 10, Resistor_SMD:R_0805_2012Metric, F.Cu at (58.1, 66.7)
- added R22: 10, Resistor_SMD:R_0805_2012Metric, F.Cu at (58.1, 69.6)
- added R23: 10, Resistor_SMD:R_0805_2012Metric, F.Cu at (58.1, 72.6)
- added R24: 1k, Resistor_SMD:R_0805_2012Metric, F.Cu at (58.1, 75.5)
- added R25: 10k, Resistor_SMD:R_0805_2012Metric, F.Cu at (62.5, 60.8)
- added R26: 10k, Resistor_SMD:R_0805_2012Metric, F.Cu at (62.5, 63.7)
- added R27: 10k, Resistor_SMD:R_0805_2012Metric, F.Cu at (62.5, 66.7)
- added R28: 1k, Resistor_SMD:R_0805_2012Metric, F.Cu at (163.4, 121.1)
- added R29: 1k, Resistor_SMD:R_0805_2012Metric, F.Cu at (163.4, 124.0)
- added R3: 3k, Resistor_SMD:R_0805_2012Metric, F.Cu at (63.1, 40.7)
- added R30: 1k, Resistor_SMD:R_0805_2012Metric, F.Cu at (163.4, 127.0)
- added R31: 1k, Resistor_SMD:R_0805_2012Metric, F.Cu at (163.4, 129.9)
- added R32: 10k, Resistor_SMD:R_0805_2012Metric, F.Cu at (163.4, 132.9)
- added R33: 10k, Connector_JST:JST_PH_B2B-PH-K_1x02_P2.00mm_Vertical, F.Cu at (145.3, 90.0)
- added R34: 10k, Resistor_SMD:R_0805_2012Metric, F.Cu at (159.4, 88.8)
- added R35: -, Resistor_SMD:R_0805_2012Metric, F.Cu at (159.4, 91.7)
- added R36: -, Resistor_SMD:R_0805_2012Metric, F.Cu at (159.4, 94.7)
- added R37: 10k, Connector_JST:JST_PH_B2B-PH-K_1x02_P2.00mm_Vertical, F.Cu at (145.3, 96.6)
- added R38: 10k, Resistor_SMD:R_0805_2012Metric, F.Cu at (159.4, 97.6)
- added R39: 10k, Connector_JST:JST_PH_B2B-PH-K_1x02_P2.00mm_Vertical, F.Cu at (145.3, 103.1)
- added R4: 500, Resistor_SMD:R_0805_2012Metric, F.Cu at (63.1, 43.7)
- added R40: 10k, Resistor_SMD:R_0805_2012Metric, F.Cu at (159.4, 100.6)
- added R41: 10k, Resistor_SMD:R_0805_2012Metric, F.Cu at (159.4, 103.5)
- added R42: 1k, Resistor_SMD:R_0805_2012Metric, F.Cu at (163.8, 88.8)
- added R43: 10k, Resistor_SMD:R_0805_2012Metric, F.Cu at (163.8, 91.7)
- added R44: 1k, Resistor_SMD:R_0805_2012Metric, F.Cu at (163.8, 94.7)
- added R45: 10k, Resistor_SMD:R_0805_2012Metric, F.Cu at (163.8, 97.6)
- added R46: 1k, Resistor_SMD:R_0805_2012Metric, F.Cu at (163.8, 100.6)
- added R47: 10k, Resistor_SMD:R_0805_2012Metric, F.Cu at (282.6, 243.7)
- added R48: 10k, Resistor_SMD:R_0805_2012Metric, F.Cu at (282.6, 246.6)
- added R49: 15k, Resistor_SMD:R_0805_2012Metric, F.Cu at (282.6, 249.6)
- added R5: 500, Resistor_SMD:R_0805_2012Metric, F.Cu at (67.5, 34.8)
- added R50: 15k, Resistor_SMD:R_0805_2012Metric, F.Cu at (282.6, 252.5)
- added R51: 10k, Resistor_SMD:R_0805_2012Metric, F.Cu at (287.0, 243.7)
- added R52: 10k, Resistor_SMD:R_0805_2012Metric, F.Cu at (287.0, 246.6)
- added R53: 10k, Resistor_SMD:R_0805_2012Metric, F.Cu at (287.0, 249.6)
- added R54: 10k, Resistor_SMD:R_0805_2012Metric, F.Cu at (287.0, 252.5)
- added R55: 10k, Resistor_SMD:R_0805_2012Metric, F.Cu at (291.4, 243.7)
- added R56: 10k, Resistor_SMD:R_0805_2012Metric, F.Cu at (291.4, 246.6)
- added R57: 10k, Resistor_SMD:R_0805_2012Metric, F.Cu at (291.4, 249.6)
- added R58: 10k, Resistor_SMD:R_0805_2012Metric, F.Cu at (291.4, 252.5)
- added R59: 10k, Resistor_SMD:R_0805_2012Metric, F.Cu at (96.2, 144.0)
- added R6: 1k, Resistor_SMD:R_0805_2012Metric, F.Cu at (67.5, 37.8)
- added R60: 10k, Resistor_SMD:R_0805_2012Metric, F.Cu at (96.2, 146.9)
- added R61: 15k, Resistor_SMD:R_0805_2012Metric, F.Cu at (96.2, 149.9)
- added R62: 15k, Resistor_SMD:R_0805_2012Metric, F.Cu at (96.2, 152.8)
- added R63: 10k, Resistor_SMD:R_0805_2012Metric, F.Cu at (100.6, 144.0)
- added R64: 10k, Resistor_SMD:R_0805_2012Metric, F.Cu at (100.6, 146.9)
- added R65: 10k, Resistor_SMD:R_0805_2012Metric, F.Cu at (100.6, 149.9)
- added R66: 10k, Resistor_SMD:R_0805_2012Metric, F.Cu at (100.6, 152.8)
- added R67: 10k, Resistor_SMD:R_0805_2012Metric, F.Cu at (105.0, 144.0)
- added R68: 10k, Resistor_SMD:R_0805_2012Metric, F.Cu at (105.0, 146.9)
- added R69: 10k, Resistor_SMD:R_0805_2012Metric, F.Cu at (105.0, 149.9)
- added R7: 10k, Resistor_SMD:R_0805_2012Metric, F.Cu at (67.5, 40.7)
- added R70: 10k, Resistor_SMD:R_0805_2012Metric, F.Cu at (105.0, 152.8)
- added R71: 10k, Resistor_SMD:R_0805_2012Metric, F.Cu at (162.3, 75.0)
- added R72: 10k, Resistor_SMD:R_0805_2012Metric, F.Cu at (162.3, 77.9)
- added R73: 15k, Resistor_SMD:R_0805_2012Metric, F.Cu at (162.3, 80.9)
- added R74: 15k, Resistor_SMD:R_0805_2012Metric, F.Cu at (162.3, 83.8)
- added R75: 10k, Resistor_SMD:R_0805_2012Metric, F.Cu at (166.7, 75.0)
- added R76: 10k, Resistor_SMD:R_0805_2012Metric, F.Cu at (166.7, 77.9)
- added R77: 10k, Resistor_SMD:R_0805_2012Metric, F.Cu at (166.7, 80.9)
- added R78: 10k, Resistor_SMD:R_0805_2012Metric, F.Cu at (166.7, 83.8)
- added R79: 10k, Resistor_SMD:R_0805_2012Metric, F.Cu at (171.1, 75.0)
- added R8: 10k, Resistor_SMD:R_0805_2012Metric, F.Cu at (67.5, 43.7)
- added R80: 10k, Resistor_SMD:R_0805_2012Metric, F.Cu at (171.1, 77.9)
- added R81: 10k, Resistor_SMD:R_0805_2012Metric, F.Cu at (171.1, 80.9)
- added R82: 10k, Resistor_SMD:R_0805_2012Metric, F.Cu at (171.1, 83.8)
- added R83: 10k, Resistor_SMD:R_0805_2012Metric, F.Cu at (129.3, 40.5)
- added R84: 10k, Resistor_SMD:R_0805_2012Metric, F.Cu at (129.3, 43.4)
- added R85: 15k, Resistor_SMD:R_0805_2012Metric, F.Cu at (129.3, 46.4)
- added R86: 15k, Resistor_SMD:R_0805_2012Metric, F.Cu at (129.3, 49.3)
- added R87: 10k, Resistor_SMD:R_0805_2012Metric, F.Cu at (133.7, 40.5)
- added R88: 10k, Resistor_SMD:R_0805_2012Metric, F.Cu at (133.7, 43.4)
- added R89: 10k, Resistor_SMD:R_0805_2012Metric, F.Cu at (133.7, 46.4)
- added R9: 1k, Resistor_SMD:R_0805_2012Metric, F.Cu at (71.9, 34.8)
- added R90: 10k, Resistor_SMD:R_0805_2012Metric, F.Cu at (133.7, 49.3)
- added R91: 10k, Resistor_SMD:R_0805_2012Metric, F.Cu at (138.1, 40.5)
- added R92: 10k, Resistor_SMD:R_0805_2012Metric, F.Cu at (138.1, 43.4)
- added R93: 10k, Resistor_SMD:R_0805_2012Metric, F.Cu at (138.1, 46.4)
- added R94: 10k, Resistor_SMD:R_0805_2012Metric, F.Cu at (138.1, 49.3)
- added R95: 10k, Resistor_SMD:R_0805_2012Metric, F.Cu at (96.2, 109.5)
- added R96: 10k, Resistor_SMD:R_0805_2012Metric, F.Cu at (96.2, 112.4)
- added R97: 15k, Resistor_SMD:R_0805_2012Metric, F.Cu at (96.2, 115.4)
- added R98: 15k, Resistor_SMD:R_0805_2012Metric, F.Cu at (96.2, 118.3)
- added R99: 10k, Resistor_SMD:R_0805_2012Metric, F.Cu at (100.6, 109.5)
- added RP1: Raspberry_Pi_2_3, Connector_PinHeader_2.54mm:PinHeader_2x20_P2.54mm_Vertical, F.Cu at (332.8, 130.6)
- added SW1: SW_DPST_x2, Button_Switch_SMD:SW_SPST_PTS647_Sx38, F.Cu at (59.4, 87.7)
- added SWD1: Conn_01x05_Socket, Connector_PinSocket_2.54mm:PinSocket_1x05_P2.54mm_Vertical, F.Cu at (42.5, 123.4)
- added U3: LM2596S-ADJ, PCM_Package_TO_SOT_SMD_AKL:TO-263-5_TabPin3_ThermalVias, F.Cu at (42.0, 49.6)
- added U6: FT232RL, Package_SO:SSOP-28_5.3x10.2mm_P0.65mm, F.Cu at (147.6, 143.2)
- added X1: 8MHz, Crystal:Crystal_HC49-U_Vertical, F.Cu at (50.4, 81.1)
- C12: value 100n -> 22n
- Q3, Q4: value MMBT3904 -> 2N7002
- U1: value STM32F405RGTx -> LM2596S-ADJ; footprint Package_QFP:LQFP-64_10x10mm_P0.5mm -> PCM_Package_TO_SOT_SMD_AKL:TO-263-5_TabPin3_ThermalVias
- U2: value FT232RL -> LM2596S-ADJ; footprint Package_SO:SSOP-28_5.3x10.2mm_P0.65mm -> PCM_Package_TO_SOT_SMD_AKL:TO-263-5_TabPin3_ThermalVias
- U4: value W5500 -> RT9193-33GB; footprint Package_QFP:LQFP-48_7x7mm_P0.5mm -> Package_TO_SOT_SMD:SOT-23-5
- U5: value W25Q32JVSS -> STM32F407VGTx; footprint Package_SO:SOIC-8_5.3x5.3mm_P1.27mm -> Package_QFP:LQFP-100_14x14mm_P0.5mm
- moved MC1 162.0 mm to (266.9, 191.8), turned to -90 degrees
- moved Q2 145.6 mm to (53.0, 86.7)
- moved Q1 145.5 mm to (48.6, 86.7), turned to 0 degrees
- moved C11 113.2 mm to (72.0, 19.8), turned to 0 degrees
- moved C12 108.3 mm to (72.0, 22.8), turned to 0 degrees
- moved U1 91.2 mm to (42.0, 24.6)
- moved U2 84.6 mm to (42.0, 37.1)
- moved U5 74.0 mm to (42.2, 68.6)
- moved Q3 73.7 mm to (159.4, 107.3), turned to 0 degrees
- moved Q4 73.7 mm to (163.8, 107.3)
- moved USB1 68.2 mm to (145.2, 127.2)
- moved U4 57.8 mm to (67.9, 54.6)
Connections:
- C11 pad 1: /Motor0/ENDSTOP_A -> GND
- C11 pad 2: GND -> +5V
- C12 pad 1: /Motor0/ENDSTOP_B -> GND
- C12 pad 2: GND -> Net-(U4-BP)
- MC1 pad 4: +5V -> EN
- Q2 pad 3: /Motor0/STEP -> EN
- Q3 pad 1: Net-(Q3-B) -> /TIM4_PWM_3
- Q3 pad 3: Net-(Q3-C) -> Net-(Q3-D)
- Q4 pad 1: Net-(Q3-C) -> /TIM8_2_TABLE_ON
- Q4 pad 3: /Motor0/DIR -> Net-(Q4-D)
- U1 pad 1: +3.3V -> +24V
- U1 pad 2: /DISP_SPI_CS1 -> Net-(D2-K)
- U1 pad 3: /ETH_INT -> GND
- U1 pad 4: /ETH_RST -> Net-(U1-FB)
- U1 pad 5: /STM32F405RG/OSC_IN -> GND
- U2 pad 1: Net-(U2-TXD) -> +24V
- U2 pad 2: unconnected-(U2-DTR-Pad2) -> Net-(D3-K)
- U2 pad 3: unconnected-(U2-RTS-Pad3) -> GND
- U2 pad 4: +3.3V -> Net-(U2-FB)
- U2 pad 5: Net-(U2-RXD) -> GND
- U4 pad 1: /W5500_module/W5500_TXN -> +5V
- U4 pad 2: /W5500_module/W5500_TXP -> GND
- U4 pad 3: GND -> +5V
- U4 pad 4: +3.3V -> Net-(U4-BP)
- U4 pad 5: /W5500_module/W5500_RXN -> +3.3V
- U5 pad 1: Net-(U5-~{CS}) -> /PIN_DIR_2
- U5 pad 2: Net-(U5-DO(IO1)) -> /PIN_DIR_3
- U5 pad 3: unconnected-(U5-IO2-Pad3) -> /PIN_DIR_4
- U5 pad 4: GND -> /PIN_DIR_5
- U5 pad 5: Net-(U5-DI(IO0)) -> /PIN_DIR_6
- U5 pad 6: Net-(U5-CLK) -> +3.3V
- U5 pad 7: unconnected-(U5-IO3-Pad7) -> /SOME_PIN_0
- U5 pad 8: +3.3V -> /SOME_PIN_1
- USB1 pad 2: Net-(U2-USBD-) -> Net-(U6-USBD-)
- USB1 pad 3: Net-(U2-USBD+) -> Net-(U6-USBD+)
Routing:
- net /Motor0/ESA: track 12.7 -> 0.00 mm
- net /Motor0/ESB: track 12.4 -> 0.00 mm
- net /Motor0/STEP: track 9.03 -> 0.00 mm
- net /Motor0/DIR: track 8.57 -> 0.00 mm
- net /Motor0/ENDSTOP_A: track 6.67 -> 0.00 mm
- net /Motor0/ENDSTOP_B: track 6.46 -> 0.00 mm
- net Net-(Q1-C): track 4.24 -> 0.00 mm
- net Net-(Q3-C): track 4.20 -> 0.00 mm
Other:
- board outline added: 56 x 86 mm

Commit message: Начал радиакально трассировать плату, вывел все порты для шаговиков
Parts:
- Q10, Q11, Q14, Q15, Q18, Q19, Q22, Q23, Q26, Q27, Q30, Q31, Q34, Q35, Q38, Q39, Q42, Q43, Q6, Q7, R100, R101, R102, R103, R104, R109, R110, R111, R112, R113, R114, R115, R116, R121, R122, R123, R124, R125, R126, R127, R128, R133, R134, R135, R136, R137, R138, R139, R140, R145, R146, R147, R148, R149, R150, R151, R152, R157, R158, R159, R160, R161, R162, R163, R164, R49, R50, R51, R52, R53, R54, R55, R56, R61, R62, R63, R64, R65, R66, R67, R68, R73, R74, R75, R76, R77, R78, R79, R80, R85, R86, R87, R88, R89, R90, R91, R92, R97, R98, R99: moved to B.Cu
- moved Q10 194.7 mm to (271.2, 172.2), turned to 180 degrees
- moved Q42 194.5 mm to (271.2, 15.2), turned to 180 degrees
- moved Q34 193.9 mm to (271.2, 54.4), turned to 180 degrees
- moved Q22 192.8 mm to (271.2, 113.3), turned to 180 degrees
- moved Q11 190.9 mm to (271.2, 175.9), turned to 180 degrees
- moved Q43 189.6 mm to (271.2, 18.9), turned to 180 degrees
- moved Q35 189.1 mm to (271.2, 58.2), turned to 180 degrees
- moved Q23 188.4 mm to (271.2, 117.0), turned to 180 degrees
- moved R60 187.4 mm to (280.2, 182.4), turned to 90 degrees
- moved C39 187.4 mm to (280.2, 187.2), turned to -90 degrees
- moved Q12 186.9 mm to (272.2, 172.2)
- moved Q44 186.7 mm to (272.2, 15.2)
- moved MC2 186.5 mm to (262.4, 174.8), turned to -90 degrees
- moved Q36 186.1 mm to (272.2, 54.4)
- moved R62 185.9 mm to (278.9, 187.1), turned to 90 degrees
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Routing:
- net EN: track 0.00 -> 354.0 mm
- net /Motor6/ESB: track 0.00 -> 38.3 mm
- net /Motor2/ESB: track 0.00 -> 38.3 mm
- net /Motor1/ESB: track 0.00 -> 38.3 mm
- net /Motor9/ESB: track 0.00 -> 38.3 mm
- net /Motor8/ESB: track 0.00 -> 38.3 mm
- net /Motor7/ESB: track 0.00 -> 38.3 mm
- net /Motor5/ESB: track 0.00 -> 38.3 mm
- net /Motor4/ESB: track 0.00 -> 38.3 mm
- net /Motor3/ESB: track 0.00 -> 38.3 mm
- net /Motor2/DIR: track 0.00 -> 30.2 mm
- net /Motor5/DIR: track 0.00 -> 30.2 mm
- net /Motor4/DIR: track 0.00 -> 30.2 mm
- net /Motor9/DIR: track 0.00 -> 30.2 mm
- net /Motor8/DIR: track 0.00 -> 30.2 mm
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Other:
- board size 56 x 86 mm -> 90.1 x 196.2 mm

Commit message: Этап трассировки полным ходом
Parts:
- C1, C2, C3, C4, C5, C6: footprint Capacitor_SMD:C_0805_2012Metric -> Capacitor_SMD:CP_Elec_6.3x7.7
- C31, LD6, LD7, R30, R31: moved to B.Cu
- moved R13 294.0 mm to (345.8, 94.6)
- moved R14 294.0 mm to (345.8, 97.5)
- moved R15 294.0 mm to (345.8, 100.5)
- moved R16 294.0 mm to (345.8, 103.5)
- moved R17 294.0 mm to (345.8, 106.4)
- moved R18 294.0 mm to (345.8, 109.3)
- moved R25 294.0 mm to (354.6, 94.6)
- moved R26 294.0 mm to (354.6, 97.5)
- moved R27 294.0 mm to (354.6, 100.5)
- moved R19 294.0 mm to (350.2, 94.6)
- moved R20 294.0 mm to (350.2, 97.5)
- moved R21 294.0 mm to (350.2, 100.5)
- moved R22 294.0 mm to (350.2, 103.5)
- moved R23 294.0 mm to (350.2, 106.4)
- moved R24 294.0 mm to (350.2, 109.3)
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Connections:
- C53 pad 1: /ES_B_9 -> /ES_B_8
- PWR1 pad 1: +24V -> GND
- PWR1 pad 2: GND -> +24V
- R101 pad 2: /TIM3_STEP_1 -> /TIM3_STEP_4
- R113 pad 2: /TIM3_STEP_2 -> /TIM3_STEP_3
- R125 pad 2: /TIM3_STEP_3 -> /TIM3_STEP_2
- R137 pad 2: /TIM3_STEP_4 -> /TIM3_STEP_1
- R144 pad 1: /ES_B_9 -> /ES_B_8
- R146 pad 2: /ES_B_9 -> /ES_B_8
- R148 pad 2: /ES_B_9 -> /ES_B_8
- U5 pad 1: /PIN_DIR_2 -> /STM32F407VG/PE2
- U5 pad 15: /ES_B_1 -> /STM32F407VG/PC0
- U5 pad 16: /ES_B_2 -> /STM32F407VG/PC1
- U5 pad 17: /ES_B_3 -> /STM32F407VG/PC2
- U5 pad 18: /ES_B_4 -> /STM32F407VG/PC3
- U5 pad 2: /PIN_DIR_3 -> /STM32F407VG/PE3
- U5 pad 3: /PIN_DIR_4 -> /STM32F407VG/PE4
- U5 pad 34: /ES_B_5 -> /STM32F407VG/PC5
- U5 pad 38: /PIN_DIR_7 -> /STM32F407VG/PE7
- U5 pad 39: /PIN_DIR_8 -> /STM32F407VG/PE8
- U5 pad 4: /PIN_DIR_5 -> /STM32F407VG/PE5
- U5 pad 40: /PIN_DIR_9 -> /STM32F407VG/PE9
- U5 pad 41: /ES_A_0 -> /STM32F407VG/PE10
- U5 pad 42: /ES_A_1 -> /STM32F407VG/PE11
- U5 pad 43: /ES_A_2 -> /STM32F407VG/PE12
- U5 pad 44: /ES_A_3 -> /STM32F407VG/PE13
- U5 pad 45: /ES_A_4 -> /STM32F407VG/PE14
- U5 pad 46: /ES_A_5 -> /STM32F407VG/PE15
- U5 pad 5: /PIN_DIR_6 -> /STM32F407VG/PE6
- U5 pad 58: /ES_A_6 -> /STM32F407VG/PD11
- U5 pad 59: /ES_A_7 -> /STM32F407VG/PD12
- U5 pad 60: /ES_A_8 -> /STM32F407VG/PD13
- U5 pad 61: /ES_A_9 -> /STM32F407VG/PD14
- U5 pad 62: /ES_B_0 -> /STM32F407VG/PD15
- U5 pad 63: /ES_B_6 -> /STM32F407VG/PC6
- U5 pad 78: /ES_B_7 -> /STM32F407VG/PC10
- U5 pad 79: /ES_B_8 -> /STM32F407VG/PC11
- U5 pad 80: /ES_B_9 -> /STM32F407VG/PC12
- U5 pad 92: /TIM4_STEP_1 -> /TIM4_PWM_4
- U5 pad 93: /TIM4_STEP_2 -> /TIM4_PWM_3
- U5 pad 95: /TIM4_PWM_3 -> /TIM4_STEP_2
- U5 pad 96: /TIM4_PWM_4 -> /TIM4_STEP_1
- U5 pad 97: /PIN_DIR_0 -> /STM32F407VG/PE0
- U5 pad 98: /PIN_DIR_1 -> /STM32F407VG/PE1
Routing:
- net +5V: track 0.00 -> 899.7 mm, vias 0 -> 11
- net EN: track 354.0 -> 23.7 mm
- net /TIM2/5_STEP_1: track 0.00 -> 123.4 mm, vias 0 -> 1
- net /TIM2/5_STEP_2: track 0.00 -> 103.5 mm, vias 0 -> 1
- net /TIM4_STEP_2: track 0.00 -> 94.9 mm, vias 0 -> 1
- net +12V: track 0.00 -> 93.8 mm
- net /TIM2/5_STEP_3: track 0.00 -> 84.1 mm, vias 0 -> 1
- net /TIM4_STEP_1: track 0.00 -> 73.0 mm, vias 0 -> 1
- net /TIM2/5_STEP_4: track 0.00 -> 70.4 mm, vias 0 -> 1
- net +3.3V: track 0.00 -> 57.8 mm, vias 0 -> 3
- net +24V: track 0.00 -> 53.2 mm
- net /TIM3_STEP_1: track 0.00 -> 41.9 mm, vias 0 -> 1
- net /TIM3_STEP_4: track 0.00 -> 39.2 mm, vias 0 -> 1
- net Net-(LD7-K): track 0.00 -> 26.8 mm, vias 0 -> 1
- net /TIM3_STEP_2: track 0.00 -> 24.1 mm, vias 0 -> 1
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Other:
- outline, holes or cut-outs redrawn
- board text added: "+12V"
- board text added: "+24V"
- board text added: "+3.3V"
- board text added: "+5V"
