File: MasterBoard.kicad_sch (KiCad schematic)
At the start: 3 parts

Commit message: Придумал название для данного поколения
Parts:
- added J1, J2, J3, J4: HX711, Connector_JST:JST_PH_B4B-PH-K_1x04_P2.00mm_Vertical, symbol Connector:Conn_01x04_Socket
Connections:
- net +5V: now also J1.1 (Pin_1), J2.1 (Pin_1), J3.1 (Pin_1), J4.1 (Pin_1)
- net GND: now also J1.4 (Pin_4), J2.4 (Pin_4), J3.4 (Pin_4), J4.4 (Pin_4)
- net RP_UART_RX: now reaches RP1.10 (GPIO15/RXD)
- net RP_BOOT0: now reaches RP1.11 (GPIO17)
- net RP_RST: now reaches RP1.12 (GPIO18/PWM0)
- net SOME_PIN_2: now reaches RP1.13 (GPIO27)
- net SPI2_MOSI: now reaches RP1.19 (MOSI0/GPIO10)
- net SPI2_MISO: now reaches RP1.21 (MISO0/GPIO9)
- net SOME_PIN_0: now reaches RP1.22 (GPIO25)
- net SPI2_SCK: now reaches RP1.23 (SCLK0/GPIO11)
- net SPI2_CS: now reaches RP1.24 (~{CE0}/GPIO8)
- net SPI2_NSS: now reaches RP1.26 (~{CE1}/GPIO7)
- net RP_UART1_TX: now reaches RP1.27 (ID_SD/GPIO0)
- net RP_UART1_RX: now reaches RP1.28 (ID_SC/GPIO1)
- net SOME_PIN_1: now reaches RP1.37 (GPIO26)
- net RP_UART_TX: now reaches RP1.8 (GPIO14/TXD)
- new net HX711_DAT_1: J1.3 (Pin_3)
- new net HX711_DAT_2: J2.3 (Pin_3)
- new net HX711_DAT_3: J3.3 (Pin_3)
- new net HX711_DAT_4: J4.3 (Pin_3)
- new net HX711_SCK_1: J1.2 (Pin_2)
- new net HX711_SCK_2: J2.2 (Pin_2)
- new net HX711_SCK_3: J3.2 (Pin_2)
- new net HX711_SCK_4: J4.2 (Pin_2)
- no-connect marks 0 -> 22
Other:
- sheet STM32F407VG ports: added none; removed PA8, PD4
- note added: "1) OctopusNode 2) KrakenNode 3) SpiderNode 4) HydraNode 5) MedusaNode"
- company: Филимонов и К -> (none)
- title: (none) -> OctopusNode

Commit message: Обновил обозначения, а то старая нумерация была специфической
Parts:
- renumbered D9800 to D1, SWD0 to SWD1
Changed lines of the file:
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@@
 		(dnp no)
 		(fields_autoplaced yes)
-		(property "Reference" "D9800"
+		(property "Reference" "D1"
 			(at 60.0075 154.94 0)
 			(effects
@@
 			(project "MasterBoard"
 				(path "/97e8f341-b455-4614-ab7f-cc310164e7aa"
-					(reference "D9800")
+					(reference "D1")
 					(unit 1)
 				)
@@
 		(dnp no)
 		(fields_autoplaced yes)
-		(property "Reference" "#PWR0368"
+		(property "Reference" "#PWR02"
 			(at 43.18 85.09 0)
 			(effects
@@
 			(project "MasterBoard"
 				(path "/97e8f341-b455-4614-ab7f-cc310164e7aa"
-					(reference "#PWR0368")
+					(reference "#PWR02")
 					(unit 1)
 				)
@@
 		(dnp no)
 		(fields_autoplaced yes)
-		(property "Reference" "#PWR0369"
+		(property "Reference" "#PWR04"
 			(at 43.18 104.14 0)
 			(effects
@@
 			(project "MasterBoard"
 				(path "/97e8f341-b455-4614-ab7f-cc310164e7aa"
-					(reference "#PWR0369")
+					(reference "#PWR04")
 					(unit 1)
 				)
@@
 		(dnp no)
 		(fields_autoplaced yes)
-		(property "Reference" "#PWR0370"
+		(property "Reference" "#PWR06"
 			(at 43.18 124.46 0)
 			(effects
@@
 			(project "MasterBoard"
 				(path "/97e8f341-b455-4614-ab7f-cc310164e7aa"
-					(reference "#PWR0370")
+					(reference "#PWR06")
 					(unit 1)
 				)
@@
 		(dnp no)
 		(fields_autoplaced yes)
-		(property "Reference" "#PWR010"
+		(property "Reference" "#PWR01"
 			(at 43.18 74.93 0)
 			(effects
@@
 			(project "MasterBoard"
 				(path "/97e8f341-b455-4614-ab7f-cc310164e7aa"
-					(reference "#PWR010")
+					(reference "#PWR01")
 					(unit 1)
 				)
@@
 		(dnp no)
 		(fields_autoplaced yes)
-		(property "Reference" "#PWR012"
+		(property "Reference" "#PWR05"
 			(at 43.18 114.3 0)
 			(effects
@@
 			(project "MasterBoard"
 				(path "/97e8f341-b455-4614-ab7f-cc310164e7aa"
-					(reference "#PWR012")
+					(reference "#PWR05")
 					(unit 1)
 				)
@@
 		(dnp no)
 		(fields_autoplaced yes)
-		(property "Reference" "#PWR0327"
+		(property "Reference" "#PWR012"
 			(at 227.33 151.13 0)
 			(effects
@@
 			(project "MasterBoard"
 				(path "/97e8f341-b455-4614-ab7f-cc310164e7aa"
-					(reference "#PWR0327")
+					(reference "#PWR012")
 					(unit 1)
 				)
@@
 		(dnp no)
 		(fields_autoplaced yes)
-		(property "Reference" "#PWR011"
+		(property "Reference" "#PWR03"
 			(at 43.18 93.98 0)
 			(effects
@@
 			(project "MasterBoard"
 				(path "/97e8f341-b455-4614-ab7f-cc310164e7aa"
-					(reference "#PWR011")
+					(reference "#PWR03")
 					(unit 1)
 				)
@@
 		(dnp no)
 		(fields_autoplaced yes)
-		(property "Reference" "#PWR09"
+		(property "Reference" "#PWR011"
 			(at 226.06 76.2 0)
 			(effects
@@
 			(project "MasterBoard"
 				(path "/97e8f341-b455-4614-ab7f-cc310164e7aa"
-					(reference "#PWR09")
+					(reference "#PWR011")
 					(unit 1)
 				)
@@
 		(dnp no)
 		(fields_autoplaced yes)
-		(property "Reference" "#PWR013"
+		(property "Reference" "#PWR07"
 			(at 43.18 133.35 0)
 			(effects
@@
 			(project "MasterBoard"
 				(path "/97e8f341-b455-4614-ab7f-cc310164e7aa"
-					(reference "#PWR013")
+					(reference "#PWR07")
 					(unit 1)
 				)
@@
 		(dnp no)
 		(fields_autoplaced yes)
-		(property "Reference" "#PWR0326"
+		(property "Reference" "#PWR013"
 			(at 228.6 76.2 0)
 			(effects
@@
 			(project "MasterBoard"
 				(path "/97e8f341-b455-4614-ab7f-cc310164e7aa"
-					(reference "#PWR0326")
+					(reference "#PWR013")
 					(unit 1)
 				)
@@
 		(dnp no)
 		(fields_autoplaced yes)
-		(property "Reference" "#PWR0371"
+		(property "Reference" "#PWR08"
 			(at 43.18 143.51 0)
 			(effects
@@
 			(project "MasterBoard"
 				(path "/97e8f341-b455-4614-ab7f-cc310164e7aa"
-					(reference "#PWR0371")
+					(reference "#PWR08")
 					(unit 1)
 				)
@@
 		(dnp no)
 		(fields_autoplaced yes)
-		(property "Reference" "#PWR0240"
+		(property "Reference" "#PWR010"
 			(at 72.39 163.83 0)
 			(effects
@@
 			(project "MasterBoard"
 				(path "/97e8f341-b455-4614-ab7f-cc310164e7aa"
-					(reference "#PWR0240")
+					(reference "#PWR010")
 					(unit 1)
 				)
@@
 		(on_board yes)
 		(dnp no)
-		(property "Reference" "SWD0"
+		(property "Reference" "SWD1"
 			(at 48.26 165.0999 0)
 			(effects
@@
 			(project ""
 				(path "/97e8f341-b455-4614-ab7f-cc310164e7aa"
-					(reference "SWD0")
+					(reference "SWD1")
 					(unit 1)
 				)
@@
 		(dnp no)
 		(fields_autoplaced yes)
-		(property "Reference" "#PWR0205"
+		(property "Reference" "#PWR09"
 			(at 58.42 179.07 0)
 			(effects
@@
 			(project "MasterBoard"
 				(path "/97e8f341-b455-4614-ab7f-cc310164e7aa"
-					(reference "#PWR0205")
-					(unit 1)
-				)
+					(reference "#PWR09")
+					(unit 1)
+				)
